File: ACE 2027/BIMU_V1_0/Controle.kicad_sch (KiCad schematic)
At the start: 32 parts, among them J201 USB_C_Receptacle_USB2.0_16P, J202 UART_connector, J203 RJ45, J204 RJ45, SW201 SW_Push, SW202 SW_Push, U201 ESP32-C3, U202 SN65HVD232DR, Y201 ABM8-40.000MHZ-10-D1G-T

Commit message: finalisation des connexions pour le BIMU. Il reste encore une révision à faire
Parts:
- added C213: 0.1μF, Capacitor_SMD:C_0603_1608Metric_Pad1.08x0.95mm_HandSolder, symbol Device:C
- added C214: 22μF, Capacitor_SMD:C_0603_1608Metric_Pad1.08x0.95mm_HandSolder, symbol Device:C
- added D202: CONNECTED LED, LED_SMD:LED_0805_2012Metric_Pad1.15x1.40mm_HandSolder, symbol Device:LED
- added R203, R204, R205, R206: 0Ω, Resistor_SMD:R_0402_1005Metric_Pad0.72x0.64mm_HandSolder, symbol Device:R_US
- added R209: 120Ω, Resistor_SMD:R_0603_1608Metric_Pad0.98x0.95mm_HandSolder, symbol Device:R_US
- D203: renamed from D202; value LED POWER -> ERROR LED
- renumbered C202 to C201, C203 to C202, C204 to C203, C205 to C204, C206 to C205, C207 to C206, C208 to C207, C209 to C208, C210 to C209, C211 to C210, C212 to C211, C213 to C212, J202 to J201, J201 to J202, R203 to R207, R204 to R208, R205 to R210, R206 to R211, R207 to R212
Connections:
- net 5V Ethernet is gone; now on net +5V: J203.7, J204.7
- net GND Ethernet is gone; now on net GND: J203.8, J204.8
- net RXD is gone; now on net TWAI_CAN_RX: U202.4 (RXD)
- net TXD is gone; now on net TWAI_CAN_TX: U202.1 (TXD)
- net +3.3V: now also U201.2 (VDD3P3), U201.3 (VDD3P3), U201.31 (VDDA), U201.32 (VDDA), C213.1, C214.1
- net ERROR_LED: now also U201.10 (MTDI/GPIO5/ADC2_CH0)
- net GND: now also C213.2, C214.2, D202.1 (K)
- net U0RX: now also U201.27 (U0RXD/GPIO20), R203.2, R206.1
- net U0TX: now also U201.28 (U0TXD/GPIO21), R204.2, R205.1
- net CONNECTED LED: now reaches U201.14 (GPIO8)
- net CONNECTED LED: now also R209.2
- net TWAI_CAN_RX: now reaches U201.4 (XTAL_32K_P/ADC1_CH0)
- net TWAI_CAN_TX: now reaches U201.5 (XTAL_32K_N/ADC1_CH1)
- net I2C_SDA: now reaches J203.3, J204.3
- net I2C_SCL: now reaches J203.4, J204.4
- net at J203.5: now also R204.1; no longer J204.5
- net at J203.6: now also R203.1; no longer J204.6
- new net: J204.5, R205.2
- new net: J204.6, R206.2
- new net: D202.2 (A), R209.1
- no-connect marks 5 -> 12
Other:
- note added: "ESP-32 CLOCK"
- moved on the sheet: C206, C207, C208, C209, D203, J201, J203, J204, R210, U201, Y201
