File: ACE 2027/BIMU_V1_0/Controle.kicad_sch (KiCad schematic)
At the start: 40 parts, among them J201 UART_connector, J202 USB_C_Receptacle_USB2.0_16P, J203 RJ45, J204 RJ45, SW201 SW_Push, SW202 SW_Push, U201 ESP32-C3, U202 SN65HVD232DR, Y201 ABM8-40.000MHZ-10-D1G-T

Commit message: Réglé les problèmes soulevé par la pull request
Parts:
- removed C202, C203, C210, C211: 0.1μF, Capacitor_SMD:C_0805_2012Metric_Pad1.18x1.45mm_HandSolder, symbol Device:C
- removed D201: USBLC6-2SC6, digikey-footprints:SOT23-6L, symbol dk_TVS-Diodes:USBLC6-2SC6
- removed U201: ESP32-C3, Package_DFN_QFN:QFN-32-1EP_5x5mm_P0.5mm_EP3.45x3.45mm, symbol Espressif:ESP32-C3
- added D204: USBLC6-2SC6, digikey-footprints:SOT23-6L, symbol BIMU_Custom:USBLC6-2SC6
- added U203: ESP32-C3, Package_DFN_QFN:QFN-32-1EP_5x5mm_P0.5mm_EP3.45x3.45mm, symbol BIMU_Custom:ESP32-C3
- SW201, SW202: footprint Button_Switch_SMD:SW_DIP_SPSTx01_Slide_6.7x4.1mm_W6.73mm_P2.54mm_LowProfile_JPin -> Button_Switch_SMD:SW_SPST_B3U-1100P-B; Digi-Key_PN (none) -> SW1021CT-ND
- renumbered C214 to C201, C213 to C202, C201 to C203, C204 to C206, C205 to C207, C206 to C208, C207 to C209, C208 to C210, C209 to C211, C212 to C214
Connections:
- net +3.3V: now also U203.2 (VDD3P3), U203.3 (VDD3P3), U203.31 (VDDA), U203.32 (VDDA)
- net +5V: now also D204.5
- net BOOT: now also U203.15 (GPIO9/BOOT)
- net CONNECTED LED: now also U203.14 (GPIO8)
- net CS: now also U203.16 (GPIO10)
- net EN: now also U203.7 (CHIP_EN)
- net ERROR_LED: now also U203.10 (MTDI/GPIO5/ADC2_CH0)
- net GND: now also D204.2, U203.33 (GND)
- net INT1: now also U203.9 (MTMS/GPIO4/ADC1_CH4)
- net INT2: now also U203.8 (GPIO3/ADC1_CH3)
- net SCL: now also U203.12 (MTCK/GPIO6)
- net SDA: now also U203.13 (MTDO/GPIO7)
- net TWAI_CAN_RX: now also U203.4 (GPIO0)
- net TWAI_CAN_TX: now also U203.5 (GPIO1)
- net U0RX: now also U203.27 (U0RXD/GPIO20)
- net U0TX: now also U203.28 (U0TXD/GPIO21)
- net USB_D+: now also D204.4, U203.25 (GPIO18/USB_D-)
- net USB_D-: now also D204.6, U203.26 (GPIO19/USB_D+)
- net XTAL_N: now also U203.29 (XTAL_N)
- net XTAL_P: now also U203.30 (XTAL_P)
- net at J202.A7 (D-), J202.B7 (D-): now also D204.1
- net at J202.A6 (D+), J202.B6 (D+): now also D204.3
- new net SDO: U203.6 (GPIO2/ADC1_CH2)
Other:
- note added: "#define IMU_PIN_SCL GPIO_NUM_5 // SPI CLK #define IMU_PIN_SDO GPIO_NUM_6 // SPI MISO #define IMU_PIN_SDA GPIO_NUM_7 // SPI MOSI #define IMU_PIN_CS GPIO_NUM_10 // Chip Select #define IMU_PIN_INT1 GPIO_NUM_4 // FIFO/Data Ready"
- note removed: "#define IMU_PIN_SCL GPIO_NUM_5 // SPI CLK #define IMU_PIN_SDX GPIO_NUM_6 // SPI MISO #define IMU_PIN_SDA GPIO_NUM_7 // SPI MOSI #define IMU_PIN_CS GPIO_NUM_10 // Chip Select #define IMU_PIN_INT1 GPIO_NUM_4 // FIFO/Data Ready"

Commit message: Réglé des petits problèmes avec la puce IMU
Parts:
- removed D204: USBLC6-2SC6, digikey-footprints:SOT23-6L, symbol BIMU_Custom:USBLC6-2SC6
- added D201: USBLC6-2SC6, digikey-footprints:SOT23-6L, symbol BIMU_Custom:USBLC6-2SC6
- R211, R212: value 60Ω -> 50Ω; Digi-Key_PN P60.4DACT-ND -> 541-CRCW080550R0FKTACT-ND
- renumbered C206 to C204, C207 to C205, C208 to C206, C209 to C207, C210 to C208, C211 to C209, C214 to C210, U203 to U201
Connections:
- net +5V: now also D201.5
- net GND: now also D201.2
- net USB_D+: now also D201.4
- net USB_D-: now also D201.6
- net at J202.A6 (D+), J202.B6 (D+): now also D201.3
- net at J202.A7 (D-), J202.B7 (D-): now also D201.1
- net SCL renamed SCLK
- net SDA renamed MOSI
- net SDO renamed MISO
Other:
- note added: "#define IMU_PIN_SCLk GPIO_NUM_5 // SPI CLK #define IMU_PIN_MISO GPIO_NUM_6 // SPI MISO #define IMU_PIN_MOSI GPIO_NUM_7 // SPI MOSI #define IMU_PIN_CS GPIO_NUM_10 // Chip Select #define IMU_PIN_INT1 GPIO_NUM_4 // FIFO/Data Ready"
- note removed: "#define IMU_PIN_SCL GPIO_NUM_5 // SPI CLK #define IMU_PIN_SDO GPIO_NUM_6 // SPI MISO #define IMU_PIN_SDA GPIO_NUM_7 // SPI MOSI #define IMU_PIN_CS GPIO_NUM_10 // Chip Select #define IMU_PIN_INT1 GPIO_NUM_4 // FIFO/Data Ready"

Commit message: mise à jours de numéro de  composants
Parts:
- J203, J204: Digi-Key_PN (none) -> 609-1046-ND
- SW201, SW202: footprint Button_Switch_SMD:SW_SPST_B3U-1100P-B -> Button_Switch_SMD:SW_SPST_B3U-1000P
Changed lines of the file:
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@@
 			)
 		)
+		(property "Digi-Key_PN" "609-1046-ND"
+			(at 81.28 116.84 0)
+			(effects
+				(font
+					(size 1.27 1.27)
+				)
+				(hide yes)
+			)
+		)
 		(pin "2"
 		)
@@
 			)
 		)
+		(property "Digi-Key_PN" "609-1046-ND"
+			(at 173.99 116.84 0)
+			(effects
+				(font
+					(size 1.27 1.27)
+				)
+				(hide yes)
+			)
+		)
 		(pin "2"
 		)
@@
 			)
 		)
-		(property "Footprint" "Button_Switch_SMD:SW_SPST_B3U-1100P-B"
+		(property "Footprint" "Button_Switch_SMD:SW_SPST_B3U-1000P"
 			(at 204.47 92.71 0)
 			(effects
@@
 			)
 		)
-		(property "Footprint" "Button_Switch_SMD:SW_SPST_B3U-1100P-B"
+		(property "Footprint" "Button_Switch_SMD:SW_SPST_B3U-1000P"
 			(at 204.47 115.57 0)
 			(effects
