File: ACE 2027/BIMU_V1_0/_autosave-Controle.kicad_sch (KiCad schematic)
At the start: 40 parts, among them J201 UART_connector, J202 USB_C_Receptacle_USB2.0_16P, J203 RJ45, J204 RJ45, SW201 SW_Push, SW202 SW_Push, U201 ESP32-C3, U202 SN65HVD232DR, Y201 ABM8-40.000MHZ-10-D1G-T

Commit message: Finalisé la révision du schéma
Parts:
- renumbered C214 to C201, C213 to C202, C201 to C203, C202 to C204, C203 to C205, C204 to C206, C205 to C207, C206 to C208, C207 to C209, C208 to C210, C209 to C211, C210 to C212, C211 to C213, C212 to C214
