File: ACE 2027/BIMU_V1_0/BIMU_V_1.kicad_pcb (KiCad board)
At the start: 2 copper layers, 35 x 40.5 mm, 53 parts, among them J201 USB_C_Receptacle_USB2.0_16P, J202 UART_connector, J203 RJ45, J204 RJ45, J301 Thermal_ResistanceM, SW201 SW_Push, SW202 SW_Push, U101 AP7361C-33E, U201 ESP32-C3, U202 SN65HVD232DR, U301 LSM6DS3, Y201 ABM8-40.000MHZ-10-D1G-T

Commit message: mise à jours de numéro de  composants
Parts:
- removed C211, C212: 0.1μF, Capacitor_SMD:C_0603_1608Metric_Pad1.08x0.95mm_HandSolder
- removed C213: 47nF, Capacitor_SMD:C_0603_1608Metric_Pad1.08x0.95mm_HandSolder
- removed J301: Thermal_ResistanceM, Connector_PinHeader_1.27mm:PinHeader_1x02_P1.27mm_Vertical
- removed R301: 10KΩ, Resistor_SMD:R_0805_2012Metric_Pad1.20x1.40mm_HandSolder
- removed R302, R303: 1.2KΩ, Resistor_SMD:R_0603_1608Metric_Pad0.98x0.95mm_HandSolder
- added C201: 22μF, Capacitor_SMD:C_0805_2012Metric_Pad1.18x1.45mm_HandSolder, F.Cu at (70.8, 39.9)
- added D203: ERROR LED, LED_SMD:LED_0805_2012Metric_Pad1.15x1.40mm_HandSolder, F.Cu at (150.1, 61.8)
- added R208: 5.1KΩ, Resistor_SMD:R_0805_2012Metric_Pad1.20x1.40mm_HandSolder, F.Cu at (75.6, 48.7)
- added R209: 330Ω, Resistor_SMD:R_0805_2012Metric_Pad1.20x1.40mm_HandSolder, F.Cu at (75.6, 51.7)
- added R210: 330Ω, Resistor_SMD:R_0805_2012Metric_Pad1.20x1.40mm_HandSolder, F.Cu at (75.6, 54.6)
- added R211: 50Ω, Resistor_SMD:R_0805_2012Metric_Pad1.20x1.40mm_HandSolder, B.Cu at (137.8, 57.7)
- added R212: 50Ω, Resistor_SMD:R_0805_2012Metric_Pad1.20x1.40mm_HandSolder, B.Cu at (132.7, 57.8)
- C103, C104, D102, D103, U101: moved to B.Cu
- C202, C203, C204, C205, C301, C302: footprint Capacitor_SMD:C_0603_1608Metric_Pad1.08x0.95mm_HandSolder -> Capacitor_SMD:C_0805_2012Metric_Pad1.18x1.45mm_HandSolder
- C206: value 0.1μF -> 12pF; footprint Capacitor_SMD:C_0603_1608Metric_Pad1.08x0.95mm_HandSolder -> Capacitor_SMD:C_0805_2012Metric_Pad1.18x1.45mm_HandSolder
- C208: value 12pF -> 0.1μF
- C209: value 0.1μF -> 22μF; footprint Capacitor_SMD:C_0603_1608Metric_Pad1.08x0.95mm_HandSolder -> Capacitor_SMD:C_0805_2012Metric_Pad1.18x1.45mm_HandSolder
- C210: value 22μF -> 47nF; moved to B.Cu
- D101: value Green_power -> POWER LED; footprint Diode_SMD:D_0805_2012Metric -> LED_SMD:LED_0805_2012Metric_Pad1.15x1.40mm_HandSolder
- D202: value LED POWER -> CONNECTED LED
- J201: value USB_C_Receptacle_USB2.0_16P -> UART_connector; footprint Connector_USB:USB_C_Receptacle_HRO_TYPE-C-31-M-12 -> Connector_PinSocket_2.54mm:PinSocket_1x04_P2.54mm_Vertical
- J202: value UART_connector -> USB_C_Receptacle_USB2.0_16P; footprint Connector_PinSocket_2.54mm:PinSocket_1x04_P2.54mm_Vertical -> Connector_USB:USB_C_Receptacle_GCT_USB4105-xx-A_16P_TopMnt_Horizontal
- R201, R202: footprint Resistor_SMD:R_0603_1608Metric_Pad0.98x0.95mm_HandSolder -> Resistor_SMD:R_0805_2012Metric_Pad1.20x1.40mm_HandSolder
- R203, R204: value 5.1KΩ -> 0Ω; footprint Resistor_SMD:R_0603_1608Metric_Pad0.98x0.95mm_HandSolder -> Resistor_SMD:R_0402_1005Metric_Pad0.72x0.64mm_HandSolder; moved to B.Cu
- R205: value 120Ω -> 0Ω; footprint Resistor_SMD:R_0603_1608Metric_Pad0.98x0.95mm_HandSolder -> Resistor_SMD:R_0402_1005Metric_Pad0.72x0.64mm_HandSolder; moved to B.Cu
- R206: value 60Ω -> 0Ω; footprint Resistor_SMD:R_0603_1608Metric_Pad0.98x0.95mm_HandSolder -> Resistor_SMD:R_0402_1005Metric_Pad0.72x0.64mm_HandSolder; moved to B.Cu
- R207: value 60Ω -> 5.1KΩ; footprint Resistor_SMD:R_0603_1608Metric_Pad0.98x0.95mm_HandSolder -> Resistor_SMD:R_0805_2012Metric_Pad1.20x1.40mm_HandSolder
- SW201, SW202: footprint Button_Switch_SMD:SW_DIP_SPSTx01_Slide_6.7x4.1mm_W6.73mm_P2.54mm_LowProfile_JPin -> Button_Switch_SMD:SW_SPST_B3U-1000P
- U301: value LSM6DS3 -> LSM6DSV16BXTR
- moved D101 88.1 mm to (150.1, 52.5)
- moved H101 82.0 mm to (148.3, 86.8)
- moved J203 74.8 mm to (139.9, 60.6), turned to 180 degrees
- moved J202 71.4 mm to (148.9, 69.8), turned to 90 degrees
- moved C210 66.2 mm to (135.5, 54.2)
- moved H102 65.0 mm to (120.7, 53.0)
- moved R204 64.3 mm to (137.1, 71.9), turned to -90 degrees
- moved R206 63.4 mm to (137.2, 68.5), turned to -90 degrees
- moved R203 62.8 mm to (135.1, 71.9), turned to -90 degrees
- moved R205 61.6 mm to (135.2, 68.5), turned to -90 degrees
- moved J204 59.7 mm to (131.2, 79.8)
- moved U101 51.9 mm to (122.6, 63.5)
- moved J201 50.0 mm to (146.1, 53.4)
- moved D202 49.5 mm to (150.1, 57.2)
- moved D103 49.4 mm to (130.8, 68.1)
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Connections:
- net Net-(J203-Pad3) renamed I2C_SDA
- net Net-(J203-Pad4) renamed I2C_SCL
- net SCL renamed SCLK
- net SDA renamed MOSI
- C202 pad 1: +5V -> +3.3V
- C203 pad 1: GND -> +5V
- C203 pad 2: USB_D- -> GND
- C204 pad 1: USB_D+ -> EN
- C205 pad 1: EN -> BOOT
- C206 pad 1: BOOT -> XTAL_P
- C207 pad 1: XTAL_P -> XTAL_N
- C208 pad 1: XTAL_N -> +3.3V
- C210 pad 1: +3.3V -> GND
- C210 pad 2: GND -> Net-(C210-Pad2)
- J203 pad 7: /Controle/5V Ethernet -> +5V
- J203 pad 8: /Controle/GND Ethernet -> GND
- J204 pad 5: Net-(J203-Pad5) -> Net-(J204-Pad5)
- J204 pad 6: Net-(J203-Pad6) -> Net-(J204-Pad6)
- J204 pad 7: /Controle/5V Ethernet -> +5V
- J204 pad 8: /Controle/GND Ethernet -> GND
- R201 pad 1: Net-(J201-CC1) -> Net-(J202-CC1)
- R202 pad 1: Net-(J201-CC2) -> Net-(J202-CC2)
- R203 pad 1: BOOT -> Net-(J203-Pad6)
- R203 pad 2: +3.3V -> U0RX
- R204 pad 1: EN -> Net-(J203-Pad5)
- R204 pad 2: +3.3V -> U0TX
- R205 pad 1: Net-(D202-A) -> U0TX
- R205 pad 2: ERROR_LED -> Net-(J204-Pad5)
- R206 pad 1: CAN_P -> U0RX
- R206 pad 2: Net-(C213-Pad2) -> Net-(J204-Pad6)
- R207 pad 1: Net-(C213-Pad2) -> BOOT
- R207 pad 2: CAN_N -> +3.3V
- U201 pad 10: unconnected-(U201-MTDI/GPIO5/ADC2_CH0-Pad10) -> ERROR_LED
- U201 pad 14: unconnected-(U201-GPIO8-Pad14) -> CONNECTED LED
- U201 pad 2: Net-(U201-VDD3P3-Pad2) -> +3.3V
- U201 pad 27: unconnected-(U201-U0RXD/GPIO20-Pad27) -> U0RX
- U201 pad 28: unconnected-(U201-U0TXD/GPIO21-Pad28) -> U0TX
- U201 pad 3: Net-(U201-VDD3P3-Pad2) -> +3.3V
- U201 pad 31: Net-(U201-VDDA-Pad31) -> +3.3V
- U201 pad 32: Net-(U201-VDDA-Pad31) -> +3.3V
- U201 pad 4: unconnected-(U201-XTAL_32K_P/ADC1_CH0-Pad4) -> TWAI_CAN_RX
- U201 pad 5: unconnected-(U201-XTAL_32K_N/ADC1_CH1-Pad5) -> TWAI_CAN_TX
- U201 pad 6: SDX -> MISO
- U202 pad 1: TXD -> TWAI_CAN_TX
- U202 pad 4: RXD -> TWAI_CAN_RX
- U301 pad 1: GND -> MISO
- U301 pad 10: unconnected-(U301-NC-Pad10) -> INT2
- U301 pad 2: SDX -> GND
- U301 pad 3: unconnected-(U301-SCX-Pad3) -> GND
- U301 pad 9: INT2 -> GND
