File: ACE 2027/BIMU/BIMU_V1_0/Controle.kicad_sch (KiCad schematic)
At the start: 36 parts, among them J201 UART_connector, J202 USB_C_Receptacle_USB2.0_16P, J203 RJ45, J204 RJ45, SW201 SW_Push, SW202 SW_Push, U201 ESP32-C3, U202 SN65HVD232DR, Y201 ABM8-40.000MHZ-10-D1G-T

Commit message: Avancement du pcb layout
Parts:
- TP201, TP202: footprint Connector_PinHeader_2.54mm:PinHeader_1x01_P2.54mm_Vertical -> TestPoint:TestPoint_Pad_1.0x1.0mm
Changed lines of the file:
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@@
 			)
 		)
-		(property "Footprint" "Connector_PinHeader_2.54mm:PinHeader_1x01_P2.54mm_Vertical"
+		(property "Footprint" "TestPoint:TestPoint_Pad_1.0x1.0mm"
 			(at 391.16 29.21 0)
 			(effects
@@
 			)
 		)
-		(property "Footprint" "Connector_PinHeader_2.54mm:PinHeader_1x01_P2.54mm_Vertical"
+		(property "Footprint" "TestPoint:TestPoint_Pad_1.0x1.0mm"
 			(at 394.97 54.61 0)
 			(effects

Commit message: Légère amélioration de la clarité des shémas électriquea
Other:
- note added: "Clock 40MHZ ±10PPM pour le ESP-32"
- note added: "Use internally for flash Do not use"
- note removed: "40MHZ ±10PPM"
- note removed: "Use internally for flash"
- moved on the sheet: C208, C209, C210, R211, R212, TP201, TP202, U202

Commit message: Fixer le problème de footprint avec le BIMU!
Parts:
- D201: footprint digikey-footprints:SOT23-6L -> BIMU:SOT23-6L
Changed lines of the file:
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@@
 			)
 		)
-		(property "Footprint" "digikey-footprints:SOT23-6L"
+		(property "Footprint" "BIMU:SOT23-6L"
 			(at 130.81 49.53 0)
 			(effects
