File: ACE 2027/BIMU/BIMU_V1_0/Controle.kicad_sch (KiCad schematic)
At the start: 36 parts, among them J201 UART_connector, J202 USB_C_Receptacle_USB2.0_16P, J203 RJ45, J204 RJ45, SW201 SW_Push, SW202 SW_Push, U201 ESP32-C3, U202 SN65HVD232DR, Y201 ABM8-40.000MHZ-10-D1G-T

Commit message: Correction inversion usb pin
Connections:
- net USB_D+: now also U201.26 (GPIO19/USB_D+); no longer U201.25 (GPIO18/USB_D-)
- net USB_D-: now also U201.25 (GPIO18/USB_D-); no longer U201.26 (GPIO19/USB_D+)
Other:
- note added: "#define IMU_PIN_SCLk GPIO_NUM_5 // SPI CLK #define IMU_PIN_MISO GPIO_NUM_6 // SPI MISO #define IMU_PIN_MOSI GPIO_NUM_7 // SPI MOSI #define IMU_PIN_CS GPIO_NUM_10 // Chip Select #define IMU_PIN_INT1 GPIO_NUM_4 // FIFO/Data Ready #define IMU_PIN_INT2 GPIO_NUM_3 // ERROR"
- note removed: "#define IMU_PIN_SCLk GPIO_NUM_5 // SPI CLK #define IMU_PIN_MISO GPIO_NUM_6 // SPI MISO #define IMU_PIN_MOSI GPIO_NUM_7 // SPI MOSI #define IMU_PIN_CS GPIO_NUM_10 // Chip Select #define IMU_PIN_INT1 GPIO_NUM_4 // FIFO/Data Ready"
Changed lines of the file:
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@@
 		)
 	)
-	(text "#define IMU_PIN_SCLk        GPIO_NUM_5    // SPI CLK\n#define IMU_PIN_MISO        GPIO_NUM_6    // SPI MISO\n#define IMU_PIN_MOSI        GPIO_NUM_7    // SPI MOSI\n#define IMU_PIN_CS          GPIO_NUM_10   // Chip Select\n#define IMU_PIN_INT1        GPIO_NUM_4    // FIFO/Data Ready"
+	(text "#define IMU_PIN_SCLk        GPIO_NUM_5    // SPI CLK\n#define IMU_PIN_MISO        GPIO_NUM_6    // SPI MISO\n#define IMU_PIN_MOSI        GPIO_NUM_7    // SPI MOSI\n#define IMU_PIN_CS          GPIO_NUM_10   // Chip Select\n#define IMU_PIN_INT1        GPIO_NUM_4    // FIFO/Data Ready\n#define IMU_PIN_INT2        GPIO_NUM_3    // ERROR"
 		(exclude_from_sim no)
 		(at 26.416 165.1 0)
@@
 	(global_label "USB_D-"
 		(shape bidirectional)
-		(at 133.35 207.01 0)
+		(at 133.35 209.55 0)
 		(fields_autoplaced yes)
 		(effects
@@
 		)
 		(property "Intersheetrefs" "${INTERSHEET_REFS}"
-			(at 145.0665 207.01 0)
+			(at 145.0665 209.55 0)
 			(hide yes)
 			(show_name no)
@@
 	(global_label "USB_D+"
 		(shape bidirectional)
-		(at 133.35 209.55 0)
+		(at 133.35 207.01 0)
 		(fields_autoplaced yes)
 		(effects
@@
 		)
 		(property "Intersheetrefs" "${INTERSHEET_REFS}"
-			(at 145.0665 209.55 0)
-			(hide yes)
-			(show_name no)
+			(at 145.0665 207.01 0)
+			(hide yes)
+			(show_name no)

Commit message: Auto stash before merge of "main" and "origin/main"
Parts:
- D201: Digi-Key_PN 497-5235-1-ND -> 4518-USBLC6-2SC6CT-ND
Changed lines of the file:
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@@
 			)
 		)
-		(property "Datasheet" "http://www.st.com/content/ccc/resource/technical/document/datasheet/06/1d/48/9c/6c/20/4a/b2/CD00050750.pdf/files/CD00050750.pdf/jcr:content/translations/en.CD00050750.pdf"
+		(property "Datasheet" "https://www.umw-ic.com/static/pdf/b2c190f0a00a742e1ffd3347f22dc112.pdf"
 			(at 130.81 46.99 0)
 			(hide yes)
@@
 			)
 		)
-		(property "Digi-Key_PN" "497-5235-1-ND"
+		(property "Digi-Key_PN" "4518-USBLC6-2SC6CT-ND"
 			(at 130.81 44.45 0)
 			(hide yes)
