File: ACE 2027/BIMU/BIMU_V1_0/BIMU_V_1.kicad_pcb (KiCad board)
At the start: 4 copper layers, 40 x 35 mm, 53 parts, among them J201 UART_connector, J202 USB_C_Receptacle_USB2.0_16P, J203 RJ45, J204 RJ45, U101 AP7361C-33E, U202 SN65HVD232DR, U301 LSM6DSV16BXTR, Y201 ABM8-40.000MHZ-10-D1G-T

Commit message: Changé pour de vrai le footprint
Parts:
- D201: footprint digikey-footprints:SOT23-6L -> BIMU:SOT23-6L
