File: ACE 2027/BIMU/BIMU_V1_0/BIMU_V_1.kicad_pcb (KiCad board)
At the start: 4 copper layers, 40 x 35 mm, 53 parts, among them J201 UART_connector, J202 USB_C_Receptacle_USB2.0_16P, J203 RJ45, J204 RJ45, U101 AP7361C-33E, U202 SN65HVD232DR, U301 LSM6DSV16BXTR, Y201 ABM8-40.000MHZ-10-D1G-T

Commit message: Correction inversion usb pin
Parts:
- renumbered POWER to D101, CONNECTED to D202, ERROR to D203, EN to SW201, BOOT to SW202, TP_GND to TP101, TP_5V to TP102, TP_3.3V to TP103, TP_CAN_P to TP201, TP_CAN_N to TP202, ESP32 to U201
Connections:
- U201 pad 25: USB_D+ -> USB_D-
- U201 pad 26: USB_D- -> USB_D+
