File: ACE 2027/daisyChainPcb_V1_0/Alimentation.kicad_sch (KiCad schematic)
At the start: 0 parts

Commit message: Electrical schematic ready for first PR
Parts:
- added C3, C4: 4.7uF, Capacitor_SMD:C_0805_2012Metric_Pad1.18x1.45mm_HandSolder, symbol Device:C_Small
- added U2: AP7361C-33E-13, daisyChain_Custom:SOT223_DIO-L, symbol daisyChain_Custom:AP7361C-33E-13
Connections:
- new net +5V: C3.1, U2.1 (IN)
- new net GND: C3.2, C4.2, U2.2 (GND), U2.4 (GND)
- new net VCC_3V3: C4.1, U2.3 (OUT)
Other:
- note added: "5V to 3.3V"
