File: ACE 2027/BMS/BMS_V1_0/BMS_V1_0.kicad_pcb (KiCad board)
At the start: 4 copper layers, 40 x 35 mm, 53 parts, among them J201 UART_connector, J202 USB_C_Receptacle_USB2.0_16P, J203 RJ45, J204 RJ45, U101 AP7361C-33E, U202 SN65HVD232DR, U301 LSM6DSV16BXTR, Y201 ABM8-40.000MHZ-10-D1G-T

Commit message: Avancement circuit sélecteur
Parts:
- removed BOOT, EN: SW_Push, Button_Switch_SMD:SW_SPST_B3U-1000P
- removed CONNECTED: CONNECTED LED, LED_SMD:LED_0805_2012Metric_Pad1.15x1.40mm_HandSolder
- removed D201: USBLC6-2SC6, digikey-footprints:SOT23-6L
- removed ERROR: ERROR LED, LED_SMD:LED_0805_2012Metric_Pad1.15x1.40mm_HandSolder
- removed ESP32: ESP32-C3, Package_DFN_QFN:QFN-32-1EP_5x5mm_P0.5mm_EP3.45x3.45mm
- removed H102: MountingHole, MountingHole:MountingHole_3.2mm_M3_ISO14580
- removed POWER: POWER LED, LED_SMD:LED_0805_2012Metric_Pad1.15x1.40mm_HandSolder
- removed R209, R210: 330Ω, Resistor_SMD:R_0805_2012Metric_Pad1.20x1.40mm_HandSolder
- removed R211, R212: 50Ω, Resistor_SMD:R_0805_2012Metric_Pad1.20x1.40mm_HandSolder
- removed TP_3.3V: TP_3v3, TestPoint:TestPoint_Pad_1.0x1.0mm
- removed TP_5V: TP_5V, TestPoint:TestPoint_Pad_1.0x1.0mm
- removed TP_CAN_N: TP_CAN_N, TestPoint:TestPoint_Pad_1.0x1.0mm
- removed TP_CAN_P: TP_CAN_P, TestPoint:TestPoint_Pad_1.0x1.0mm
- removed TP_GND: TP_GND_IN, TestPoint:TestPoint_Pad_1.0x1.0mm
- added C303: 0.1uF, Capacitor_SMD:C_0805_2012Metric, F.Cu at (200.0, 89.4)
- added C401: 0.1uF, Capacitor_SMD:C_0805_2012Metric, F.Cu at (161.0, 104.4)
- added C601: 0,1µF, Capacitor_SMD:C_0805_2012Metric, F.Cu at (209.3, 49.4)
- added C602: 0.1uF, Capacitor_SMD:C_0805_2012Metric, F.Cu at (209.3, 52.4)
- added D101: POWER LED, LED_SMD:LED_0805_2012Metric_Pad1.15x1.40mm_HandSolder, F.Cu at (161.2, 101.3)
- added D202: CONNECTED LED, LED_SMD:LED_0805_2012Metric_Pad1.15x1.40mm_HandSolder, F.Cu at (153.4, 63.6)
- added D203: ERROR LED, LED_SMD:LED_0805_2012Metric_Pad1.15x1.40mm_HandSolder, F.Cu at (153.4, 66.7)
- added D301: POWER LED, LED_SMD:LED_0805_2012Metric_Pad1.15x1.40mm_HandSolder, F.Cu at (200.3, 60.4)
- added D302: BZV55B15, Diode_SMD:D_MiniMELF, F.Cu at (201.0, 83.2)
- added D303: POWER LED, LED_SMD:LED_0805_2012Metric_Pad1.15x1.40mm_HandSolder, F.Cu at (204.8, 73.6)
- added D401: BZV55B15, Diode_SMD:D_MiniMELF, F.Cu at (169.4, 99.9)
- added D402: BZV55B15, Diode_SMD:D_MiniMELF, F.Cu at (169.4, 103.2)
- added D601: BZV55B15, Diode_SMD:D_MiniMELF, F.Cu at (210.3, 46.2)
- added D602: POWER LED, LED_SMD:LED_0805_2012Metric_Pad1.15x1.40mm_HandSolder, F.Cu at (214.2, 36.5)
- added J103: Jambe_gauche, Connector_AMASS:AMASS_XT30PW-F_1x02_P2.50mm_Horizontal, F.Cu at (156.2, 87.1)
- added J104: Jambe_droite, Connector_AMASS:AMASS_XT30PW-F_1x02_P2.50mm_Horizontal, F.Cu at (171.5, 87.1)
- added Q301: NTR2101P, Package_TO_SOT_SMD:SOT-23, F.Cu at (204.7, 87.1)
- added Q401: NTR2101P, Package_TO_SOT_SMD:SOT-23, F.Cu at (184.2, 83.2)
- added Q403: NTR2101P, Package_TO_SOT_SMD:SOT-23, F.Cu at (184.2, 87.6)
- added Q601: NTR2101P, Package_TO_SOT_SMD:SOT-23, F.Cu at (214.0, 50.1)
- added R301: 330Ω, Resistor_SMD:R_0805_2012Metric_Pad1.20x1.40mm_HandSolder, F.Cu at (200.3, 63.4)
- added R302: ???Ω, Resistor_SMD:R_0805_2012Metric_Pad1.20x1.40mm_HandSolder, F.Cu at (191.0, 73.5)
- added R303: ???Ω, Resistor_SMD:R_0805_2012Metric_Pad1.20x1.40mm_HandSolder, F.Cu at (191.0, 76.5)
- added R304: ???Ω, Resistor_SMD:R_0805_2012Metric_Pad1.20x1.40mm_HandSolder, F.Cu at (191.0, 79.4)
- added R305: ???Ω, Resistor_SMD:R_0805_2012Metric_Pad1.20x1.40mm_HandSolder, F.Cu at (191.0, 82.4)
- added R306: ???Ω, Resistor_SMD:R_2512_6332Metric_Pad1.40x3.35mm_HandSolder, F.Cu at (197.9, 74.5)
- added R307: ???, Resistor_SMD:R_0805_2012Metric, F.Cu at (195.6, 78.5)
- added R308: ???Ω, Resistor_SMD:R_0805_2012Metric, F.Cu at (195.6, 81.4)
- added R309: 100Ω, Resistor_SMD:R_0805_2012Metric, F.Cu at (195.6, 84.4)
- added R401: ???Ω, Resistor_SMD:R_0805_2012Metric_Pad1.20x1.40mm_HandSolder, F.Cu at (153.4, 94.3)
- added R402: ???Ω, Resistor_SMD:R_0805_2012Metric_Pad1.20x1.40mm_HandSolder, F.Cu at (153.4, 97.3)
- added R403: ???Ω, Resistor_SMD:R_0805_2012Metric_Pad1.20x1.40mm_HandSolder, F.Cu at (153.4, 100.2)
- added R404: ???Ω, Resistor_SMD:R_0805_2012Metric_Pad1.20x1.40mm_HandSolder, F.Cu at (153.4, 103.2)
- added R405: ???, Resistor_SMD:R_0805_2012Metric, F.Cu at (178.3, 91.4)
- added R406: ???Ω, Resistor_SMD:R_0805_2012Metric, F.Cu at (178.3, 94.3)
- added R407: 100Ω, Resistor_SMD:R_0805_2012Metric, F.Cu at (178.3, 97.3)
- added R601: ???Ω, Resistor_SMD:R_0805_2012Metric_Pad1.20x1.40mm_HandSolder, F.Cu at (200.3, 36.5)
- added R602: ???Ω, Resistor_SMD:R_0805_2012Metric_Pad1.20x1.40mm_HandSolder, F.Cu at (200.3, 39.4)
- added R603: ???Ω, Resistor_SMD:R_0805_2012Metric_Pad1.20x1.40mm_HandSolder, F.Cu at (200.3, 42.4)
- added R604: ???Ω, Resistor_SMD:R_0805_2012Metric_Pad1.20x1.40mm_HandSolder, F.Cu at (200.3, 45.3)
- added R605: ???Ω, Resistor_SMD:R_2512_6332Metric_Pad1.40x3.35mm_HandSolder, F.Cu at (207.2, 37.5)
- added R606: ???, Resistor_SMD:R_0805_2012Metric, F.Cu at (204.9, 41.4)
- added R607: ???Ω, Resistor_SMD:R_0805_2012Metric, F.Cu at (204.9, 44.3)
- added R608: 100Ω, Resistor_SMD:R_0805_2012Metric, F.Cu at (204.9, 47.3)
- added SW201: SW_Push, Button_Switch_SMD:SW_SPST_B3U-1000P, F.Cu at (189.4, 57.0)
- added SW202: SW_Push, Button_Switch_SMD:SW_SPST_B3U-1000P, F.Cu at (189.4, 61.3)
- added TP101: TP_GND_IN, TestPoint:TestPoint_Pad_1.0x1.0mm, F.Cu at (157.3, 91.4)
- added TP102: TP_5V, TestPoint:TestPoint_Pad_1.0x1.0mm, F.Cu at (157.3, 94.5)
- added TP103: TP_3v3, TestPoint:TestPoint_Pad_1.0x1.0mm, F.Cu at (157.3, 97.5)
- added TP201: TP_CAN_P, TestPoint:TestPoint_Pad_1.0x1.0mm, F.Cu at (193.8, 56.3)
- added TP202: TP_CAN_N, TestPoint:TestPoint_Pad_1.0x1.0mm, F.Cu at (193.8, 59.4)
- added TP301: TP_Current, TestPoint:TestPoint_Pad_1.0x1.0mm, F.Cu at (190.1, 85.4)
- added TP302: TP_Voltage, TestPoint:TestPoint_Pad_1.0x1.0mm, F.Cu at (190.1, 88.4)
- added TP401: TP_Voltage, TestPoint:TestPoint_Pad_1.0x1.0mm, F.Cu at (157.3, 100.6)
- added TP601: TP_Current, TestPoint:TestPoint_Pad_1.0x1.0mm, F.Cu at (199.5, 48.3)
- added TP602: TP_Voltage, TestPoint:TestPoint_Pad_1.0x1.0mm, F.Cu at (199.5, 51.4)
- added U201: ESP32-S3, Package_DFN_QFN:QFN-56-1EP_7x7mm_P0.4mm_EP4x4mm, F.Cu at (181.8, 59.4)
- added U601: INA240A2PW, Package_SO:TSSOP-8_4.4x3mm_P0.65mm, F.Cu at (211.5, 42.2)
- C103, C104, C201, C202, C203, C204, C205, C210, D102, D103, R101, R201, R202, U101, U202: moved to F.Cu
- C301: value 0.1μF -> 4,7µF; moved to F.Cu
- C302: value 0.1μF -> 0,1µF; footprint Capacitor_SMD:C_0805_2012Metric_Pad1.18x1.45mm_HandSolder -> Capacitor_SMD:C_0805_2012Metric; moved to F.Cu
- J203: value RJ45 -> MoBo
- J204: value RJ45 -> BIMU
- R203, R204: value 0Ω -> 5.1KΩ; footprint Resistor_SMD:R_0402_1005Metric_Pad0.72x0.64mm_HandSolder -> Resistor_SMD:R_0805_2012Metric_Pad1.20x1.40mm_HandSolder; moved to F.Cu
- R205, R206: value 0Ω -> 330Ω; footprint Resistor_SMD:R_0402_1005Metric_Pad0.72x0.64mm_HandSolder -> Resistor_SMD:R_0805_2012Metric_Pad1.20x1.40mm_HandSolder; moved to F.Cu
- R207, R208: value 5.1KΩ -> 50Ω
- U301: value LSM6DSV16BXTR -> INA240A2PW; footprint Package_LGA:LGA-14_3x2.5mm_P0.5mm_LayoutBorder3x4y -> Package_SO:TSSOP-8_4.4x3mm_P0.65mm
- moved R101 63.6 mm to (153.4, 91.4)
- moved R201 59.3 mm to (158.2, 36.5)
- moved R202 56.1 mm to (158.2, 39.4)
- moved R205 55.0 mm to (158.2, 48.3), turned to 0 degrees
- moved R206 54.9 mm to (158.2, 51.2), turned to 0 degrees
- moved C203 53.8 mm to (153.4, 42.5), turned to 0 degrees
- moved H101 46.9 mm to (179.6, 102.3)
- moved C104 44.1 mm to (162.5, 97.3), turned to 0 degrees
- moved C201 39.7 mm to (153.4, 36.5), turned to 0 degrees
- moved C202 38.9 mm to (153.4, 39.5), turned to 0 degrees
- moved J204 38.7 mm to (182.8, 39.8)
- moved J201 36.3 mm to (162.9, 57.1)
- moved J203 36.1 mm to (165.1, 39.8), turned to 0 degrees
- moved C206 35.9 mm to (153.4, 51.6), turned to 0 degrees
- moved J202 35.9 mm to (171.0, 60.1), turned to 0 degrees
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Connections:
- C301 pad 1: +3.3V -> unconnected-(C301-Pad1)
- C301 pad 2: GND -> unconnected-(C301-Pad2)
- C302 pad 1: GND -> +3.3V
- C302 pad 2: +3.3V -> GND
- J203 pad 3: I2C_SDA -> GND
- J203 pad 4: I2C_SCL -> GND
- J203 pad 5: Net-(J203-Pad5) -> +5V
- J203 pad 6: Net-(J203-Pad6) -> +5V
- J204 pad 3: I2C_SDA -> unconnected-(J204-Pad3)
- J204 pad 4: I2C_SCL -> unconnected-(J204-Pad4)
- J204 pad 5: Net-(J204-Pad5) -> unconnected-(J204-Pad5)
- J204 pad 6: Net-(J204-Pad6) -> unconnected-(J204-Pad6)
- R203 pad 1: Net-(J203-Pad6) -> BOOT
- R203 pad 2: U0RX -> +3.3V
- R204 pad 1: Net-(J203-Pad5) -> EN
- R204 pad 2: U0TX -> +3.3V
- R205 pad 1: U0TX -> Net-(D202-A)
- R205 pad 2: Net-(J204-Pad5) -> CONNECTED LED
- R206 pad 1: U0RX -> Net-(D203-A)
- R206 pad 2: Net-(J204-Pad6) -> ERROR_LED
- R207 pad 1: BOOT -> CAN_P
- R207 pad 2: +3.3V -> Net-(C210-Pad2)
- R208 pad 1: EN -> Net-(C210-Pad2)
- R208 pad 2: +3.3V -> CAN_N
- U301 pad 1: MISO -> GND
- U301 pad 2: GND -> Net-(Q301-D)
- U301 pad 3: GND -> /Alimentation/Battery_Out_Gauche
- U301 pad 4: INT1 -> GND
- U301 pad 6: GND -> +3.3V
- U301 pad 8: +3.3V -> Current_Sense_Gauche
Routing:
- net U0RX: track 89.6 -> 0.00 mm
- net U0TX: track 86.5 -> 0.00 mm, vias 2 -> 0
- net +5V: track 73.2 -> 0.00 mm, vias 9 -> 0
- net GND: track 52.3 -> 0.00 mm, vias 49 -> 0
- net CAN_P: track 39.1 -> 0.00 mm, vias 1 -> 0
- net +3.3V: track 38.4 -> 0.00 mm, vias 27 -> 0
- net CAN_N: track 36.7 -> 0.00 mm, vias 1 -> 0
- net CONNECTED LED: track 36.1 -> 0.00 mm, vias 3 -> 0
- net EN: track 32.4 -> 0.00 mm, vias 3 -> 0
- net BOOT: track 30.5 -> 0.00 mm, vias 5 -> 0
- net ERROR_LED: track 30.3 -> 0.00 mm, vias 3 -> 0
- net USB_D+: track 26.0 -> 0.00 mm, vias 4 -> 0
- net USB_D-: track 25.7 -> 0.00 mm, vias 4 -> 0
- net CS: track 20.1 -> 0.00 mm
- net I2C_SDA: track 19.5 -> 0.00 mm, vias 2 -> 0
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- removed copper zone on In1.Cu, net +3.3V
- removed copper zone on In2.Cu, net GND
Other:
- board outline removed
- board text removed: "Conception: Josserand-Pierre Gay Vérification: Samuel Savaria"
- board text removed: "ETH-UART"
- board text removed: "MASTER"
- board text removed: "MASTER SIDE"
- board text removed: "TMB"
