File: ACE 2027/BMS/BMS_V1_0/Battery_Sub_Circuit.kicad_sch (KiCad schematic)
At the start: 12 parts, among them Q1 NTR2101P, Q2 NPN, SW1 E-STOP, SW2 RESET_SWITCH

Commit message: Avancement circuit de sécurité
Parts:
- removed C106: 4,7µF, Capacitor_SMD:C_0805_2012Metric_Pad1.18x1.45mm_HandSolder, symbol Device:C
- removed R104: ???Ω, Resistor_SMD:R_0805_2012Metric_Pad1.20x1.40mm_HandSolder, symbol Device:R_US
- added C2: 0,1µF, Capacitor_SMD:C_0805_2012Metric, symbol Device:C
- added C3: 0.1uF, Capacitor_SMD:C_0805_2012Metric, symbol Device:C
- added F1: Fuse, symbol Device:Fuse
- added R1: ???Ω, Resistor_SMD:R_2512_6332Metric_Pad1.40x3.35mm_HandSolder, symbol Device:R_US
- added R5: 100Ω, Resistor_SMD:R_0805_2012Metric, symbol Device:R_US
- added R6: ???Ω, Resistor_SMD:R_0805_2012Metric, symbol Device:R_US
- added R7: ???, Resistor_SMD:R_0805_2012Metric, symbol Device:R_US
- added U3: INA240A2PW, Package_SO:TSSOP-8_4.4x3mm_P0.65mm, symbol Amplifier_Current:INA240A2PW
Connections:
- net Battery_P: now also F1.1; no longer Q1.2 (S), R103.2
- net at Q1.3 (D), SW1.1: now also R1.1, U3.2 (+)
- net GND: now reaches Q2.3 (E), R105.1
- net GND: now also D106.1 (K), C2.2, C3.2, R6.1, U3.1 (GND), U3.4 (GND), U3.7 (REF1)
- net at D106.2 (A): now also R5.2, R6.2, R7.1
- new net: F1.2, Q1.2 (S), R103.2
- new net Battery out: R1.2, R7.2, U3.3 (-)
- new net Current sense: U3.8
- new net ESP32 supply: C2.1, U3.5 (V+), U3.6 (REF2)
- new net Voltage sense: C3.1, R5.1
Other:
- moved on the sheet: D106

Commit message: Avancement général du schémas
Parts:
- renumbered C2 to C501, C3 to C502, D1 to D501, D106 to D502, F1 to F501, Q1 to Q501, Q2 to Q502, R103 to R501, R105 to R502, R107 to R503, R106 to R504, R1 to R505, R7 to R506, R6 to R507, R5 to R508, SW2 to SW501, SW1 to SW502, U3 to U501
Connections:
- net ESP32 supply renamed +3.3V
Other:
- note added: "CURRENT SENSE"
- note added: "EMF AND E-STOP"
- note added: "VOLTAGE SENSE"
- moved on the sheet: C501, U501

Commit message: Amélioration de la présentation
Parts:
- removed SW502: E-STOP, symbol Switch:SW_Omron_B3FS
- added SW303: E-STOP, symbol Switch:SW_Omron_B3FS
- added TP301: TP_Current, TestPoint:TestPoint_Pad_1.0x1.0mm, symbol Connector:TestPoint
- added TP302: TP_Voltage, TestPoint:TestPoint_Pad_1.0x1.0mm, symbol Connector:TestPoint
- renumbered C501 to C302, C502 to C303, D501 to D302, D502 to D303, F501 to F301, Q501 to Q301, Q502 to Q302, R501 to R302, R502 to R303, R503 to R304, R504 to R305, R505 to R306, R506 to R307, R507 to R308, R508 to R309, SW501 to SW301, U501 to U301
Connections:
- net Current sense: now also TP301.1
- net Voltage sense: now also TP302.1
- net at Q301.3 (D), R306.1, U301.2 (+): now also R305.2
- net at R305.1, SW301.2 (B): now also SW303.1; no longer R304.1
- new net: R304.1, SW303.2
Other:
- moved on the sheet: R305, SW301

Commit message: Petite révision suite à une rencontre avec Olivier
Parts:
- removed F301: Fuse, symbol Device:Fuse
Connections:
- net Battery_P: now also Q301.2 (S), R302.2
Changed lines of the file:
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@@
 	(wire
 		(pts
-			(xy 29.21 125.73) (xy 36.83 125.73)
+			(xy 29.21 125.73) (xy 90.17 125.73)
 		)
 		(stroke
@@
 	(wire
 		(pts
-			(xy 44.45 125.73) (xy 90.17 125.73)
-		)
-		(stroke
-			(width 0)
-			(type default)
-		)
-	)
-	(wire
-		(pts
 			(xy 219.71 147.32) (xy 219.71 152.4)
 		)
@@
 					(unit 1)
 				)
-			)
-		)
-	)
-	(symbol
-		(lib_id "Device:Fuse")
-		(at 40.64 125.73 90)
-		(unit 1)
-		(body_style 1)
-		(exclude_from_sim no)
-		(in_bom yes)
-		(on_board yes)
-		(in_pos_files yes)
-		(dnp no)
-		(fields_autoplaced yes)
-		(property "Reference" "F301"
-			(at 40.64 119.38 90)
-			(show_name no)
-			(do_not_autoplace no)
-			(effects
-				(font
-					(size 1.27 1.27)
-				)
-			)
-		)
-		(property "Value" "Fuse"
-			(at 40.64 121.92 90)
-			(show_name no)
-			(do_not_autoplace no)
-			(effects
-				(font
-					(size 1.27 1.27)
-				)
-			)
-		)
-		(property "Footprint" ""
-			(at 40.64 127.508 90)
-			(hide yes)
-			(show_name no)
-			(do_not_autoplace no)
-			(effects
-				(font
-					(size 1.27 1.27)
-				)
-			)
-		)
-		(property "Datasheet" ""
-			(at 40.64 125.73 0)
-			(hide yes)
-			(show_name no)
-			(do_not_autoplace no)
-			(effects
-				(font
-					(size 1.27 1.27)
-				)
-			)
-		)
-		(property "Description" "Fuse"
-			(at 40.64 125.73 0)
-			(hide yes)
-			(show_name no)
-			(do_not_autoplace no)
-			(effects
-				(font
-					(size 1.27 1.27)
-				)
-			)
-		)
-		(property "Category" ""
-			(at 40.64 125.73 90)
-			(hide yes)
-			(show_name no)
-			(do_not_autoplace no)
-			(effects
-				(font
-					(size 1.27 1.27)
-				)
-			)
-		)
-		(property "DK_Datasheet_Link" ""
-			(at 40.64 125.73 90)
-			(hide yes)
-			(show_name no)
-			(do_not_autoplace no)
-			(effects
-				(font
-					(size 1.27 1.27)
-				)
-			)
-		)
-		(property "DK_Detail_Page" ""
-			(at 40.64 125.73 90)
-			(hide yes)
-			(show_name no)
-			(do_not_autoplace no)
-			(effects
-				(font
-					(size 1.27 1.27)
-				)
-			)
-		)
-		(property "Description_1" ""
-			(at 40.64 125.73 90)
-			(hide yes)
-			(show_name no)
-			(do_not_autoplace no)
-			(effects
-				(font
-					(size 1.27 1.27)
-				)
-			)
-		)
-		(property "Family" ""
-			(at 40.64 125.73 90)
-			(hide yes)
-			(show_name no)
-			(do_not_autoplace no)
-			(effects
-				(font
-					(size 1.27 1.27)
-				)
-			)
-		)
-		(property "Link" ""
-			(at 40.64 125.73 90)
-			(hide yes)
-			(show_name no)
-			(do_not_autoplace no)
-			(effects
-				(font
-					(size 1.27 1.27)
-				)
-			)
-		)
-		(property "MPN" ""
-			(at 40.64 125.73 90)
-			(hide yes)
-			(show_name no)
-			(do_not_autoplace no)
-			(effects
-				(font
-					(size 1.27 1.27)
-				)
-			)
-		)
-		(property "Manufacturer" ""
-			(at 40.64 125.73 90)
-			(hide yes)
-			(show_name no)
-			(do_not_autoplace no)
-			(effects
-				(font
-					(size 1.27 1.27)
-				)
-			)
-		)
-		(property "Status" ""
-			(at 40.64 125.73 90)
-			(hide yes)
-			(show_name no)
-			(do_not_autoplace no)
-			(effects
-				(font
-					(size 1.27 1.27)
-				)
-			)
-		)
-		(pin "2"
-		)
-		(pin "1"
-		)
-		(instances
-			(project "BMS_V1_0"
-				(path "/abeb93ed-b9ef-4503-99a7-3fce380ff294/6937e765-eead-4ea7-ba07-6590a34338ab/3082eddd-1090-4e43-a4f9-15043173df44"
-					(reference "F301")
-					(unit 1)
-				)
-				(path "/abeb93ed-b9ef-4503-99a7-3fce380ff294/6937e765-eead-4ea7-ba07-6590a34338ab/37ad5e6c-60b7-45e9-975c-2deedeb98e1a"
-					(reference "F601")
-					(unit 1)
-				)

Commit message: Avancement circuit sélecteur
Changed lines of the file:
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@@
+	)
+	(junction
+		(at 110.49 62.23)
+		(diameter 0)
+		(color 0 0 0 0)
 	)
 	(junction
@@
 	)
 	(junction
-		(at 110.49 62.23)
-		(diameter 0)
-		(color 0 0 0 0)
-	)
-	(junction
 		(at 219.71 147.32)
 		(diameter 0)
@@
 	(wire
 		(pts
-			(xy 53.34 62.23) (xy 110.49 62.23)
+			(xy 29.21 62.23) (xy 110.49 62.23)
 		)
 		(stroke
@@
 	(hierarchical_label "Battery_N"
 		(shape input)
-		(at 52.07 62.23 180)
+		(at 29.21 62.23 180)
 		(effects
 			(font
