File: ACE 2027/BMS/BMS_V1_0/Alimentation.kicad_sch (KiCad schematic)
At the start: 5 parts

Commit message: Schémas de protection avancée
Other:
- added sheet Battery_Sub_Circuit (Battery_Sub_Circuit.kicad_sch)

Commit message: Avancement circuit de sécurité
Other:
- sheet Battery_Sub_Circuit renamed Battery_Sub_Circuit_Gauche
- added sheet Battery_Sub_Circuit_Droite (Battery_Sub_Circuit.kicad_sch)
- sheet Battery_Sub_Circuit_Gauche ports: added Battery out, Battery_N, Battery_P, Current sense, Voltage sense; removed none
Changed lines of the file:
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@@
 	(sheet
 		(at 100.33 67.31)
-		(size 147.32 72.39)
+		(size 67.31 53.34)
 		(exclude_from_sim no)
 		(in_bom yes)
@@
 			(color 0 0 0 0)
 		)
-		(property "Sheetname" "Battery_Sub_Circuit"
+		(property "Sheetname" "Battery_Sub_Circuit_Gauche"
 			(at 100.33 66.5984 0)
 			(show_name no)
@@
 		)
 		(property "Sheetfile" "Battery_Sub_Circuit.kicad_sch"
-			(at 100.33 140.2846 0)
+			(at 100.33 121.2346 0)
 			(show_name no)
 			(do_not_autoplace no)
@@
 			)
 		)
+		(pin "Battery out" input
+			(at 167.64 80.01 0)
+			(effects
+				(font
+					(size 1.27 1.27)
+				)
+				(justify right)
+			)
+		)
+		(pin "Battery_N" input
+			(at 100.33 107.95 180)
+			(effects
+				(font
+					(size 1.27 1.27)
+				)
+				(justify left)
+			)
+		)
+		(pin "Battery_P" input
+			(at 100.33 80.01 180)
+			(effects
+				(font
+					(size 1.27 1.27)
+				)
+				(justify left)
+			)
+		)
+		(pin "Current sense" input
+			(at 167.64 93.98 0)
+			(effects
+				(font
+					(size 1.27 1.27)
+				)
+				(justify right)
+			)
+		)
+		(pin "Voltage sense" input
+			(at 167.64 107.95 0)
+			(effects
+				(font
+					(size 1.27 1.27)
+				)
+				(justify right)
+			)
+		)
 		(instances
 			(project "BMS_V1_0"
@@
 				)
 			)
+		)
+	)
+	(sheet
+		(at 100.33 142.24)
+		(size 67.31 53.34)
+		(exclude_from_sim no)
+		(in_bom yes)
+		(on_board yes)
+		(dnp no)
+		(fields_autoplaced yes)
+		(stroke
+			(width 0.1524)
+			(type solid)
+		)
+		(fill
+			(color 0 0 0 0)
+		)
+		(property "Sheetname" "Battery_Sub_Circuit_Droite"
+			(at 100.33 141.5284 0)
+			(show_name no)
+			(do_not_autoplace no)
+			(effects
+				(font
+					(size 1.27 1.27)
+				)
+				(justify left bottom)
+			)
+		)
+		(property "Sheetfile" "Battery_Sub_Circuit.kicad_sch"
+			(at 100.33 196.1646 0)
+			(show_name no)
+			(do_not_autoplace no)
+			(effects
+				(font
+					(size 1.27 1.27)
+				)
+				(justify left top)
+			)
+		)
+		(pin "Battery out" input
+			(at 167.64 154.94 0)
+			(effects
+				(font
+					(size 1.27 1.27)
+				)
+				(justify right)
+			)
+		)
+		(pin "Battery_N" input
+			(at 100.33 182.88 180)
+			(effects
+				(font
+					(size 1.27 1.27)
+				)
+				(justify left)
+			)
+		)
+		(pin "Battery_P" input
+			(at 100.33 154.94 180)
+			(effects
+				(font
+					(size 1.27 1.27)
+				)
+				(justify left)
+			)
+		)
+		(pin "Current sense" input
+			(at 167.64 168.91 0)
+			(effects
+				(font
+					(size 1.27 1.27)
+				)
+				(justify right)
+			)
+		)
+		(pin "Voltage sense" input
+			(at 167.64 182.88 0)
+			(effects
+				(font
+					(size 1.27 1.27)
+				)
+				(justify right)
+			)
+		)
+		(instances
+			(project "BMS_V1_0"
+				(path "/abeb93ed-b9ef-4503-99a7-3fce380ff294/6937e765-eead-4ea7-ba07-6590a34338ab"
+					(page "6")
+				)
+			)

Commit message: Avancement général du schémas
Parts:
- added C402, C403: 4,7µF, Capacitor_SMD:C_0805_2012Metric_Pad1.18x1.45mm_HandSolder, symbol Device:C
- added C404, C405: 1nF, Capacitor_SMD:C_1812_4532Metric_Pad1.57x3.40mm_HandSolder, symbol Device:C
- added D403, D404: STPS1H100A, symbol Device:D
- added D405: POWER LED, LED_SMD:LED_0805_2012Metric_Pad1.15x1.40mm_HandSolder, symbol Device:LED
- added D406, D407: BAV99, Package_TO_SOT_SMD:SOT-23, symbol Diode:BAV99
- added R402: 330Ω, Resistor_SMD:R_0805_2012Metric_Pad1.20x1.40mm_HandSolder, symbol Device:R_US
- added TP401: TP_GND_IN, TestPoint:TestPoint_Pad_1.0x1.0mm, symbol Connector:TestPoint
- added TP402: TP_5V, TestPoint:TestPoint_Pad_1.0x1.0mm, symbol Connector:TestPoint
- added TP403: TP_3v3, TestPoint:TestPoint_Pad_1.0x1.0mm, symbol Connector:TestPoint
- added U401: AP7361C-33E, Package_TO_SOT_SMD:SOT-223-3_TabPin2, symbol Regulator_Linear:AP7361C-33E
- gave numbers to parts that had none: 1
- renumbered C105 to C401, D104 to D401, D105 to D402, R102 to R401
Connections:
- new net: D403.1 (K), D404.1 (K)
- new net: D405.2 (A), R402.2
- new net +3.3V: C403.2, C404.1, C405.1, D406.2 (A), D407.2 (A), R402.1, TP403.1, U401.3 (VO)
- new net +5V: C402.2, TP402.1, U401.1 (VI)
- new net Battery_Out_Droite: D404.2 (A)
- new net Battery_Out_Gauche: D403.2 (A)
- new net CAN_N: D407.3 (K)
- new net CAN_P: D406.3 (K)
- new net GND: C402.1, C403.1, C404.2, C405.2, D405.1 (K), D406.1 (K), D407.1 (K), TP401.1, U401.2 (GND)
Other:
- note added: "1A MAX CURRENT"
- note added: "5V TO 3.3V CONVERTER"
- note added: "ALIMENTATION TO 48V"
- note added: "ALIMENTATION TO 5V"
- note added: "ESD Protection"
- note added: "MAGIE NOIR QUI PASSE DE ALIMENTATION A 5V"

Commit message: Amélioration de la présentation
Parts:
- removed C401: 4,7µF, Capacitor_SMD:C_0805_2012Metric_Pad1.18x1.45mm_HandSolder, symbol Device:C
- removed D401: POWER LED, LED_SMD:LED_0805_2012Metric_Pad1.15x1.40mm_HandSolder, symbol Device:LED
- removed D402: BAV99, Package_TO_SOT_SMD:SOT-23, symbol Diode:BAV99
- removed R401: 330Ω, Resistor_SMD:R_0805_2012Metric_Pad1.20x1.40mm_HandSolder, symbol Device:R_US
- added F101, F102, F103, F104, F105: Fuse, symbol Device:Fuse
- added J101: Batterie_gauche, symbol Connector:Conn_01x02_Pin
- added J102: Batterie_droite, symbol Connector:Conn_01x02_Pin
- added J103: Jambe_gauche, Connector_AMASS:AMASS_XT30PW-F_1x02_P2.50mm_Horizontal, symbol Connector:Conn_01x02_Pin
- added J104: Jambe_droite, Connector_AMASS:AMASS_XT30PW-F_1x02_P2.50mm_Horizontal, symbol Connector:Conn_01x02_Pin
- renumbered C402 to C101, C403 to C102, C404 to C103, C405 to C104, D405 to D101, D406 to D102, D407 to D103, D403 to D104, D404 to D105, H401 to H101, R402 to R101, TP401 to TP101, TP402 to TP102, TP403 to TP103, U401 to U101
Connections:
- net +5V: now also F105.2
- net Battery_Sub_Circuit_Droite/Battery_N: now also J102.1 (Pin_1)
- net Battery_Sub_Circuit_Droite/Battery_P: now also F102.2
- net Battery_Sub_Circuit_Gauche/Battery_N: now also J101.1 (Pin_1)
- net Battery_Sub_Circuit_Gauche/Battery_P: now also F101.2
- net GND: now also J103.1 (Pin_1), J104.1 (Pin_1)
- new net: F103.1, J103.2 (Pin_2)
- new net: F102.1, J102.2 (Pin_2)
- new net: F104.1, J104.2 (Pin_2)
- new net: F101.1, J101.2 (Pin_2)
- new net +48V: F103.2, F104.2
Other:
- note added: "CONNECTEURS OUTPUT"
- note added: "Le 5 volt sort par les ports ethernets"
- note added: "SELECTION CIRCUIT"
- moved on the sheet: C101, C102, C103, C104, D101, D102, D103, D104, D105, H101, R101, TP101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

Commit message: Avancement circuit sélecteur
Parts:
- added C401: 0.1uF, Capacitor_SMD:C_0805_2012Metric, symbol Device:C
- added D401, D402: BZV55B15, Diode_SMD:D_MiniMELF, symbol Diode:BZV55B15
- added Q401, Q403: NTR2101P, Package_TO_SOT_SMD:SOT-23, symbol Transistor_FET:NTR2101P
- added Q402, Q404: NPN, symbol Simulation_SPICE:NPN
- added R401, R402, R403, R404: ???Ω, Resistor_SMD:R_0805_2012Metric_Pad1.20x1.40mm_HandSolder, symbol Device:R_US
- added R405: ???, Resistor_SMD:R_0805_2012Metric, symbol Device:R_US
- added R406: ???Ω, Resistor_SMD:R_0805_2012Metric, symbol Device:R_US
- added R407: 100Ω, Resistor_SMD:R_0805_2012Metric, symbol Device:R_US
- added TP401: TP_Voltage, TestPoint:TestPoint_Pad_1.0x1.0mm, symbol Connector:TestPoint
Connections:
- net Battery_Out_Droite: now also Q403.2 (S), R403.2
- net Battery_Out_Gauche: now also Q401.2 (S), R401.2
- net GND: now also C401.2, Q402.3 (E), Q404.3 (E), R402.1, R404.1, R406.1
- new net: R405.1, R406.2, R407.2
- new net: D401.2 (A), Q401.1 (G), R401.1
- new net: D402.1 (K), Q404.1 (C)
- new net: D402.2 (A), Q403.1 (G), R403.1
- new net: D401.1 (K), Q402.1 (C)
- new net: Q402.2 (B), R402.2
- new net: Q404.2 (B), R404.2
- new net Sortie_Selecteur: Q401.3 (D), Q403.3 (D), R405.2
- new net Voltage_Sense_Selecteur: C401.1, R407.1, TP401.1
Other:
- note added: "CIRCUIT SELECTION"
- note added: "Ce transistor tire vers le ground pour Alumé le mosfet"
- note added: "Cette résistance force la gate à high (donc le courant ne circule pas)"
- note added: "Drain"
- note added: "Gate"
- note added: "La flêche pointe vers la source besoin d'un Vgs négatif pour fermé Si la gate est moins hautes que la source elle ouvre"
- note added: "Pull down pour ouvrir le transistor rapidement Peut-être pas requis dans ce cas si"
- note added: "Source"
- note added: "VOLTAGE SENSE"
- note removed: "SELECTION CIRCUIT"

Commit message: légère modification
Connections:
- net Circuit_selection_Gauche: now reaches Q402.2 (B), R402.2
- net Circuit_selection_Droite: now reaches Q404.2 (B), R404.2
Changed lines of the file:
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@@
+	)
+	(junction
+		(at 139.7 209.55)
+		(diameter 0)
+		(color 0 0 0 0)
 	)
 	(junction
@@
 		(pts
 			(xy 63.5 247.65) (xy 78.74 247.65)
+		)
+		(stroke
+			(width 0)
+			(type default)
+		)
+	)
+	(wire
+		(pts
+			(xy 139.7 209.55) (xy 139.7 213.36)
 		)
 		(stroke
@@
 			)
 			(justify left bottom)
+		)
+	)
+	(global_label "Circuit_selection_Gauche"
+		(shape input)
+		(at 96.52 209.55 0)
+		(fields_autoplaced yes)
+		(effects
+			(font
+				(size 1.27 1.27)
+			)
+			(justify left)
+		)
+		(property "Intersheetrefs" "${INTERSHEET_REFS}"
+			(at 123.1513 209.55 0)
+			(hide yes)
+			(show_name no)
+			(do_not_autoplace no)
+			(effects
+				(font
+					(size 1.27 1.27)
+				)
+				(justify left)
+			)
 		)
 	)
@@
 			)
 		)
+	)
+	(global_label "Circuit_selection_Droite"
+		(shape input)
+		(at 139.7 213.36 180)
+		(fields_autoplaced yes)
+		(effects
+			(font
+				(size 1.27 1.27)
+			)
+			(justify right)
+		)
+		(property "Intersheetrefs" "${INTERSHEET_REFS}"
+			(at 114.3386 213.36 0)
+			(hide yes)
+			(show_name no)
+			(do_not_autoplace no)
+			(effects
+				(font
+					(size 1.27 1.27)
+				)
+				(justify right)
+			)
+		)
