File: ACE 2027/BMS/BMS_V1_0/Capteur.kicad_sch (KiCad schematic)
At the start: 3 parts

Commit message: Avancement général du schémas
Parts:
- renumbered C303 to C301

Commit message: légère modification
Parts:
- removed C301: 4,7µF, Capacitor_SMD:C_0805_2012Metric_Pad1.18x1.45mm_HandSolder, symbol Device:C
- removed D301: POWER LED, LED_SMD:LED_0805_2012Metric_Pad1.15x1.40mm_HandSolder, symbol Device:LED
- removed R301: 330Ω, Resistor_SMD:R_0805_2012Metric_Pad1.20x1.40mm_HandSolder, symbol Device:R_US
