File: ACE 2027/daisyChainPcb/daisyChainPcb_V1_0/Controle.kicad_sch (KiCad schematic)
At the start: 20 parts, among them J1 RJ45, J2 RJ45, J3 Pads, J5 XT30, J6 XT30, J7 Pads, J8 Pads

Commit message: Fixer les numéro de composant
Parts:
- renumbered J8 to J201, J6 to J202, J5 to J203, J3 to J204, J7 to J205, J1 to J206, J2 to J207, R1 to R201, R2 to R202, TP1 to TP201, TP3 to TP202, TP2 to TP203, TP4 to TP204, TP5 to TP205, TP7 to TP206, TP6 to TP207, TP8 to TP208, TP9 to TP209, TP10 to TP210, TP11 to TP211
Changed lines of the file:
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@@
 		(dnp no)
 		(fields_autoplaced yes)
-		(property "Reference" "J1"
+		(property "Reference" "J206"
 			(at 198.12 68.58 0)
 			(show_name no)
@@
 			(project "daisyChainPcb_V1_0"
 				(path "/c963cec3-4702-49ad-9d19-390ec91e9467/cd13e174-6d34-4da6-82aa-10931bd92064"
-					(reference "J1")
+					(reference "J206")
 					(unit 1)
 				)
@@
 		(dnp no)
 		(fields_autoplaced yes)
-		(property "Reference" "TP10"
+		(property "Reference" "TP210"
 			(at 116.84 70.3579 0)
 			(show_name no)
@@
 			(project "daisyChainPcb_V1_0"
 				(path "/c963cec3-4702-49ad-9d19-390ec91e9467/cd13e174-6d34-4da6-82aa-10931bd92064"
-					(reference "TP10")
+					(reference "TP210")
 					(unit 1)
 				)
@@
 		(dnp no)
 		(fields_autoplaced yes)
-		(property "Reference" "TP4"
+		(property "Reference" "TP204"
 			(at 38.1 91.9479 0)
 			(show_name no)
@@
 			(project "daisyChainPcb_V1_0"
 				(path "/c963cec3-4702-49ad-9d19-390ec91e9467/cd13e174-6d34-4da6-82aa-10931bd92064"
-					(reference "TP4")
+					(reference "TP204")
 					(unit 1)
 				)
@@
 		(dnp no)
 		(fields_autoplaced yes)
-		(property "Reference" "#PWR03"
+		(property "Reference" "#PWR0201"
 			(at 57.15 100.33 0)
 			(hide yes)
@@
 			(project "daisyChainPcb_V1_0"
 				(path "/c963cec3-4702-49ad-9d19-390ec91e9467/cd13e174-6d34-4da6-82aa-10931bd92064"
-					(reference "#PWR03")
+					(reference "#PWR0201")
 					(unit 1)
 				)
@@
 		(dnp no)
 		(fields_autoplaced yes)
-		(property "Reference" "TP8"
+		(property "Reference" "TP208"
 			(at 78.74 91.9479 0)
 			(show_name no)
@@
 			(project "daisyChainPcb_V1_0"
 				(path "/c963cec3-4702-49ad-9d19-390ec91e9467/cd13e174-6d34-4da6-82aa-10931bd92064"
-					(reference "TP8")
+					(reference "TP208")
 					(unit 1)
 				)
@@
 		(in_pos_files yes)
 		(dnp no)
-		(property "Reference" "#PWR01"
+		(property "Reference" "#PWR0203"
 			(at 227.33 68.58 0)
 			(hide yes)
@@
 			(project "daisyChainPcb_V1_0"
 				(path "/c963cec3-4702-49ad-9d19-390ec91e9467/cd13e174-6d34-4da6-82aa-10931bd92064"
-					(reference "#PWR01")
+					(reference "#PWR0203")
 					(unit 1)
 				)
@@
 		(dnp no)
 		(fields_autoplaced yes)
-		(property "Reference" "TP2"
+		(property "Reference" "TP203"
 			(at 38.1 72.8979 0)
 			(show_name no)
@@
 			(project "daisyChainPcb_V1_0"
 				(path "/c963cec3-4702-49ad-9d19-390ec91e9467/cd13e174-6d34-4da6-82aa-10931bd92064"
-					(reference "TP2")
+					(reference "TP203")
 					(unit 1)
 				)
@@
 		(dnp no)
 		(fields_autoplaced yes)
-		(property "Reference" "J7"
+		(property "Reference" "J205"
 			(at 140.97 26.67 90)
 			(show_name no)
@@
 			(project "daisyChainPcb_V1_0"
 				(path "/c963cec3-4702-49ad-9d19-390ec91e9467/cd13e174-6d34-4da6-82aa-10931bd92064"
-					(reference "J7")
+					(reference "J205")
 					(unit 1)
 				)
@@
 		(dnp no)
 		(fields_autoplaced yes)
-		(property "Reference" "TP11"
+		(property "Reference" "TP211"
 			(at 118.11 95.7579 0)
 			(show_name no)
@@
 			(project "daisyChainPcb_V1_0"
 				(path "/c963cec3-4702-49ad-9d19-390ec91e9467/cd13e174-6d34-4da6-82aa-10931bd92064"
-					(reference "TP11")
+					(reference "TP211")
 					(unit 1)
 				)
@@
 		(dnp no)
 		(fields_autoplaced yes)
-		(property "Reference" "TP5"
+		(property "Reference" "TP205"
 			(at 62.23 72.8979 0)
 			(show_name no)
@@
 			(project "daisyChainPcb_V1_0"
 				(path "/c963cec3-4702-49ad-9d19-390ec91e9467/cd13e174-6d34-4da6-82aa-10931bd92064"
-					(reference "TP5")
+					(reference "TP205")
 					(unit 1)
 				)
@@
 		(dnp no)
 		(fields_autoplaced yes)
-		(property "Reference" "#PWR013"
+		(property "Reference" "#PWR0202"
 			(at 95.25 78.74 0)
 			(hide yes)
@@
 			(project "daisyChainPcb_V1_0"
 				(path "/c963cec3-4702-49ad-9d19-390ec91e9467/cd13e174-6d34-4da6-82aa-10931bd92064"
-					(reference "#PWR013")
+					(reference "#PWR0202")
 					(unit 1)
 				)
@@
 		(in_pos_files yes)
 		(dnp no)
-		(property "Reference" "R2"
+		(property "Reference" "R202"
 			(at 243.84 33.0199 0)
 			(show_name no)
@@
 			(project "daisyChainPcb_V1_0"
 				(path "/c963cec3-4702-49ad-9d19-390ec91e9467/cd13e174-6d34-4da6-82aa-10931bd92064"
-					(reference "R2")
+					(reference "R202")
 					(unit 1)
 				)
@@
 		(dnp no)
 		(fields_autoplaced yes)
-		(property "Reference" "J3"
+		(property "Reference" "J204"
 			(at 128.27 31.1149 90)
 			(show_name no)
@@
 			(project "daisyChainPcb_V1_0"
 				(path "/c963cec3-4702-49ad-9d19-390ec91e9467/cd13e174-6d34-4da6-82aa-10931bd92064"
-					(reference "J3")
+					(reference "J204")
 					(unit 1)
 				)
@@
 		(dnp no)
 		(fields_autoplaced yes)
-		(property "Reference" "TP1"
+		(property "Reference" "TP201"
 			(at 24.13 72.8979 0)
 			(show_name no)
@@
 			(project "daisyChainPcb_V1_0"
 				(path "/c963cec3-4702-49ad-9d19-390ec91e9467/cd13e174-6d34-4da6-82aa-10931bd92064"
-					(reference "TP1")
+					(reference "TP201")
 					(unit 1)
 				)
@@
 		(dnp no)
 		(fields_autoplaced yes)
-		(property "Reference" "#FLG02"
+		(property "Reference" "#FLG0201"
 			(at 95.25 76.835 0)
 			(hide yes)
@@
 			(project "daisyChainPcb_V1_0"
 				(path "/c963cec3-4702-49ad-9d19-390ec91e9467/cd13e174-6d34-4da6-82aa-10931bd92064"
-					(reference "#FLG02")
+					(reference "#FLG0201")
 					(unit 1)
 				)
@@
 		(dnp no)
 		(fields_autoplaced yes)
-		(property "Reference" "TP9"
+		(property "Reference" "TP209"
 			(at 102.87 70.3579 0)
 			(show_name no)
@@
 			(project "daisyChainPcb_V1_0"
 				(path "/c963cec3-4702-49ad-9d19-390ec91e9467/cd13e174-6d34-4da6-82aa-10931bd92064"
-					(reference "TP9")
+					(reference "TP209")
 					(unit 1)
 				)
@@
 		(dnp no)
 		(fields_autoplaced yes)
-		(property "Reference" "J2"
+		(property "Reference" "J207"
 			(at 273.05 68.58 0)
 			(show_name no)
@@
 			(project "daisyChainPcb_V1_0"
 				(path "/c963cec3-4702-49ad-9d19-390ec91e9467/cd13e174-6d34-4da6-82aa-10931bd92064"
-					(reference "J2")
+					(reference "J207")
 					(unit 1)
 				)
@@
 		(dnp no)
 		(fields_autoplaced yes)
-		(property "Reference" "J8"
+		(property "Reference" "J201"
 			(at 35.56 27.3049 90)
 			(show_name no)
@@
 			(project "daisyChainPcb_V1_0"
 				(path "/c963cec3-4702-49ad-9d19-390ec91e9467/cd13e174-6d34-4da6-82aa-10931bd92064"
-					(reference "J8")
+					(reference "J201")
 					(unit 1)
 				)
@@
 		(dnp no)
 		(fields_autoplaced yes)
-		(property "Reference" "R1"
+		(property "Reference" "R201"
 			(at 232.41 33.0199 0)
 			(show_name no)
@@
 			(project "daisyChainPcb_V1_0"
 				(path "/c963cec3-4702-49ad-9d19-390ec91e9467/cd13e174-6d34-4da6-82aa-10931bd92064"
-					(reference "R1")
+					(reference "R201")
 					(unit 1)
 				)
@@
 		(dnp no)
 		(fields_autoplaced yes)
-		(property "Reference" "TP3"
+		(property "Reference" "TP202"
 			(at 24.13 91.9479 0)
 			(show_name no)
@@
 			(project "daisyChainPcb_V1_0"
 				(path "/c963cec3-4702-49ad-9d19-390ec91e9467/cd13e174-6d34-4da6-82aa-10931bd92064"
-					(reference "TP3")
+					(reference "TP202")
 					(unit 1)
 				)
@@
 		(dnp no)
 		(fields_autoplaced yes)
-		(property "Reference" "TP6"
+		(property "Reference" "TP207"
 			(at 76.2 72.8979 0)
 			(show_name no)
@@
 			(project "daisyChainPcb_V1_0"
 				(path "/c963cec3-4702-49ad-9d19-390ec91e9467/cd13e174-6d34-4da6-82aa-10931bd92064"
-					(reference "TP6")
+					(reference "TP207")
 					(unit 1)
 				)
@@
 		(dnp no)
 		(fields_autoplaced yes)
-		(property "Reference" "J6"
+		(property "Reference" "J202"
 			(at 59.69 27.3049 90)
 			(show_name no)
@@
 			(project "daisyChainPcb_V1_0"
 				(path "/c963cec3-4702-49ad-9d19-390ec91e9467/cd13e174-6d34-4da6-82aa-10931bd92064"
-					(reference "J6")
+					(reference "J202")
 					(unit 1)
 				)
@@
 		(dnp no)
 		(fields_autoplaced yes)
-		(property "Reference" "J5"
+		(property "Reference" "J203"
 			(at 71.12 27.3049 90)
 			(show_name no)
@@
 			(project "daisyChainPcb_V1_0"
 				(path "/c963cec3-4702-49ad-9d19-390ec91e9467/cd13e174-6d34-4da6-82aa-10931bd92064"
-					(reference "J5")
+					(reference "J203")
 					(unit 1)
 				)
@@
 		(dnp no)
 		(fields_autoplaced yes)
-		(property "Reference" "TP7"
+		(property "Reference" "TP206"
 			(at 64.77 91.9479 0)
 			(show_name no)
@@
 			(project "daisyChainPcb_V1_0"
 				(path "/c963cec3-4702-49ad-9d19-390ec91e9467/cd13e174-6d34-4da6-82aa-10931bd92064"
-					(reference "TP7")
-					(unit 1)
-				)
+					(reference "TP206")
+					(unit 1)
+				)

Commit message: Ready for PCB PR
Connections:
- net 48V is gone; now on net +48V: J201.2 (Pin_2), J202.2 (Pin_2), J203.2 (Pin_2)
Other:
- moved on the sheet: J202, J203
