File: ACE 2027/BIMU/BIMU_V_1_1/BIMU_V_1_1.kicad_pcb (KiCad board)
At the start: 4 copper layers, 40 x 35 mm, 56 parts, among them J201 UART_connector, J202 USB_C_Receptacle_USB2.0_16P, J203 RJ45, J204 RJ45, SW201 SW_Push, SW202 SW_Push, SW203 SW_CAN, U101 AP7361C-33E, U201 ESP32-C3, U202 SN65HVD232DR, U301 LSM6DSV16BXTR, Y201 ABM8-40.000MHZ-10-D1G-T

Commit message: Mise à jour des traces pour TX et RX
Connections:
- U201 pad 4: TWAI_CAN_RX -> TWAI_CAN_TX
- U201 pad 5: TWAI_CAN_TX -> TWAI_CAN_RX
- U202 pad 1: TWAI_CAN_RX -> TWAI_CAN_TX
- U202 pad 4: TWAI_CAN_TX -> TWAI_CAN_RX
Routing:
- net TWAI_CAN_TX: track 3.09 -> 3.64 mm
- net TWAI_CAN_RX: track 3.64 -> 3.09 mm
- net +5V: vias 6 -> 5
Changed lines of the file:
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@@
 			(layers "F.Cu" "F.Mask" "F.Paste")
 			(roundrect_rratio 0.25)
-			(net "TWAI_CAN_RX")
+			(net "TWAI_CAN_TX")
 			(pinfunction "GPIO0_4")
 			(pintype "bidirectional")
@@
 			(layers "F.Cu" "F.Mask" "F.Paste")
 			(roundrect_rratio 0.25)
-			(net "TWAI_CAN_TX")
+			(net "TWAI_CAN_RX")
 			(pinfunction "GPIO1_5")
 			(pintype "bidirectional")
@@
 			(layers "B.Cu" "B.Mask" "B.Paste")
 			(roundrect_rratio 0.25)
-			(net "TWAI_CAN_RX")
+			(net "TWAI_CAN_TX")
 			(pinfunction "TXD_1")
 			(pintype "input")
@@
 			(layers "B.Cu" "B.Mask" "B.Paste")
 			(roundrect_rratio 0.25)
-			(net "TWAI_CAN_TX")
+			(net "TWAI_CAN_RX")
 			(pinfunction "RXD_4")
 			(pintype "output")
@@
 	)
 	(via
-		(at 198.06 81.51)
-		(size 0.6)
-		(drill 0.3)
-		(layers "F.Cu" "B.Cu")
-		(net "+5V")
-	)
-	(via
 		(at 201.78 60.46)
 		(size 0.6)
@@
 	)
 	(segment
-		(start 205.2 72.28)
-		(end 205.6 72.28)
-		(width 0.25)
-		(layer "F.Cu")
-		(net "+5V_USB")
-	)
-	(segment
 		(start 205.6 72.28)
 		(end 205.922792 72.28)
@@
 	)
 	(segment
-		(start 178.482475 70.7375)
-		(end 179.028966 71.283991)
-		(width 0.2)
-		(layer "F.Cu")
-		(net "TWAI_CAN_RX")
-	)
-	(segment
-		(start 177.8875 70.7375)
-		(end 178.482475 70.7375)
-		(width 0.2)
-		(layer "F.Cu")
-		(net "TWAI_CAN_RX")
-	)
-	(segment
-		(start 179.028966 71.283991)
-		(end 179.028966 71.900652)
+		(start 178.7175 70.2375)
+		(end 178.73 70.225)
 		(width 0.2)
 		(layer "F.Cu")
@@
 	)
 	(segment
-		(start 177.95 70.8)
-		(end 177.8875 70.7375)
+		(start 177.8875 70.2375)
+		(end 178.7175 70.2375)
 		(width 0.2)
 		(layer "F.Cu")
@@
 	)
 	(via
-		(at 179.028966 71.900652)
+		(at 178.73 70.225)
 		(size 0.6)
 		(drill 0.3)
@@
 	)
 	(segment
-		(start 179.733314 72.605)
-		(end 180.3 72.605)
+		(start 178.73 70.090158)
+		(end 180.025158 68.795)
 		(width 0.2)
 		(layer "B.Cu")
@@
 	)
 	(segment
-		(start 179.028966 71.900652)
-		(end 179.733314 72.605)
+		(start 178.73 70.225)
+		(end 178.73 70.090158)
 		(width 0.2)
 		(layer "B.Cu")
@@
 	)
 	(segment
-		(start 178.7175 70.2375)
-		(end 178.73 70.225)
+		(start 180.025158 68.795)
+		(end 180.3 68.795)
+		(width 0.2)
+		(layer "B.Cu")
+		(net "TWAI_CAN_RX")
+	)
+	(segment
+		(start 178.482475 70.7375)
+		(end 179.028966 71.283991)
 		(width 0.2)
 		(layer "F.Cu")
@@
 	)
 	(segment
-		(start 177.8875 70.2375)
-		(end 178.7175 70.2375)
+		(start 177.8875 70.7375)
+		(end 178.482475 70.7375)
 		(width 0.2)
 		(layer "F.Cu")
 		(net "TWAI_CAN_TX")
 	)
-	(via
-		(at 178.73 70.225)
-		(size 0.6)
-		(drill 0.3)
-		(layers "F.Cu" "B.Cu")
+	(segment
+		(start 179.028966 71.283991)
+		(end 179.028966 71.900652)
+		(width 0.2)
+		(layer "F.Cu")
 		(net "TWAI_CAN_TX")
 	)
 	(segment
-		(start 178.73 70.090158)
-		(end 180.025158 68.795)
+		(start 177.95 70.8)
+		(end 177.8875 70.7375)
 		(width 0.2)
-		(layer "B.Cu")
+		(layer "F.Cu")
+		(net "TWAI_CAN_TX")
+	)
+	(via
+		(at 179.028966 71.900652)
+		(size 0.6)
+		(drill 0.3)
+		(layers "F.Cu" "B.Cu")
 		(net "TWAI_CAN_TX")
 	)
 	(segment
-		(start 178.73 70.225)
-		(end 178.73 70.090158)
+		(start 179.733314 72.605)
+		(end 180.3 72.605)
 		(width 0.2)
 		(layer "B.Cu")
@@
 	)
 	(segment
-		(start 180.025158 68.795)
-		(end 180.3 68.795)
+		(start 179.028966 71.900652)
+		(end 179.733314 72.605)
 		(width 0.2)
 		(layer "B.Cu")
