File: ACE 2027/BIMU/BIMU_V_1_1/Controle.kicad_sch (KiCad schematic)
At the start: 36 parts, among them J201 UART_connector, J202 USB_C_Receptacle_USB2.0_16P, J203 RJ45, J204 RJ45, SW201 SW_Push, SW202 SW_Push, U201 ESP32-C3, U202 SN65HVD232DR, Y201 ABM8-40.000MHZ-10-D1G-T

Commit message: Rajouté une switch demandé par Éloi
Parts:
- added SW203: SW_CAN, Button_Switch_SMD:SW_SPDT_CK_JS102011SAQN, symbol Switch:SW_SPDT
Connections:
- net CAN_N: now also SW203.1 (A); no longer R212.2
- new net: R212.2, SW203.2 (B)
- no-connect marks 10 -> 11
Other:
- moved on the sheet: TP202
Changed lines of the file:
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@@
 	)
 	(junction
+		(at 359.41 74.93)
+		(diameter 0)
+		(color 0 0 0 0)
+	)
+	(junction
 		(at 215.9 97.79)
 		(diameter 0)
@@
 	)
 	(junction
-		(at 351.79 55.88)
+		(at 351.79 74.93)
 		(diameter 0)
 		(color 0 0 0 0)
@@
 		(color 0 0 0 0)
 	)
-	(junction
-		(at 356.87 55.88)
-		(diameter 0)
-		(color 0 0 0 0)
-	)
 	(no_connect
 		(at 77.47 245.11)
@@
 	)
 	(no_connect
+		(at 354.33 67.31)
+	)
+	(no_connect
 		(at 77.47 252.73)
 	)
@@
 	(wire
 		(pts
+			(xy 359.41 74.93) (xy 365.76 74.93)
+		)
+		(stroke
+			(width 0)
+			(type default)
+		)
+	)
+	(wire
+		(pts
 			(xy 132.08 107.95) (xy 132.08 111.76)
 		)
@@
 	(wire
 		(pts
-			(xy 349.25 55.88) (xy 351.79 55.88)
+			(xy 349.25 74.93) (xy 351.79 74.93)
 		)
 		(stroke
@@
 	(wire
 		(pts
+			(xy 359.41 67.31) (xy 359.41 74.93)
+		)
+		(stroke
+			(width 0)
+			(type default)
+		)
+	)
+	(wire
+		(pts
 			(xy 132.08 119.38) (xy 132.08 123.19)
 		)
@@
 	(wire
 		(pts
+			(xy 356.87 53.34) (xy 356.87 57.15)
+		)
+		(stroke
+			(width 0)
+			(type default)
+		)
+	)
+	(wire
+		(pts
 			(xy 209.55 120.65) (xy 215.9 120.65)
 		)
@@
 	(wire
 		(pts
-			(xy 356.87 55.88) (xy 356.87 53.34)
-		)
-		(stroke
-			(width 0)
-			(type default)
-		)
-	)
-	(wire
-		(pts
 			(xy 99.06 124.46) (xy 91.44 124.46)
 		)
@@
 	(wire
 		(pts
-			(xy 349.25 49.53) (xy 349.25 55.88)
+			(xy 349.25 49.53) (xy 349.25 74.93)
 		)
 		(stroke
@@
 	(wire
 		(pts
-			(xy 351.79 55.88) (xy 356.87 55.88)
-		)
-		(stroke
-			(width 0)
-			(type default)
-		)
-	)
-	(wire
-		(pts
 			(xy 138.43 66.04) (xy 138.43 62.23)
 		)
@@
 	(wire
 		(pts
-			(xy 356.87 55.88) (xy 365.76 55.88)
+			(xy 351.79 74.93) (xy 359.41 74.93)
 		)
 		(stroke
@@
 	(global_label "CAN_N"
 		(shape input)
-		(at 365.76 55.88 0)
+		(at 365.76 74.93 0)
 		(fields_autoplaced yes)
 		(effects
@@
 		)
 		(property "Intersheetrefs" "${INTERSHEET_REFS}"
-			(at 374.7324 55.88 0)
+			(at 374.7324 74.93 0)
 			(hide yes)
 			(show_name no)
@@
 	(symbol
 		(lib_id "Connector:TestPoint")
-		(at 351.79 55.88 180)
+		(at 351.79 74.93 180)
 		(unit 1)
 		(body_style 1)
@@
 		(dnp yes)
 		(property "Reference" "TP202"
-			(at 353.695 63.5 0)
+			(at 353.695 82.55 0)
 			(show_name no)
 			(do_not_autoplace no)
@@
 		)
 		(property "Value" "TP_CAN_N"
-			(at 354.965 60.96 0)
+			(at 354.965 80.01 0)
 			(show_name no)
 			(do_not_autoplace no)
@@
 		)
 		(property "Footprint" "TestPoint:TestPoint_Pad_1.0x1.0mm"
-			(at 346.71 55.88 0)
+			(at 346.71 74.93 0)
 			(hide yes)
 			(show_name no)
@@
 		)
 		(property "Datasheet" ""
-			(at 346.71 55.88 0)
+			(at 346.71 74.93 0)
 			(hide yes)
 			(show_name no)
@@
 		)
 		(property "Description" "test point"
-			(at 351.79 55.88 0)
+			(at 351.79 74.93 0)
 			(hide yes)
 			(show_name no)
@@
 					(unit 1)
 				)
+			)
+		)
+	)
+	(symbol
+		(lib_id "Switch:SW_SPDT")
+		(at 356.87 62.23 270)
+		(unit 1)
+		(body_style 1)
+		(exclude_from_sim no)
+		(in_bom yes)
+		(on_board yes)
+		(in_pos_files yes)
+		(dnp no)
+		(fields_autoplaced yes)
+		(property "Reference" "SW203"
+			(at 361.95 60.9599 90)
+			(show_name no)
+			(do_not_autoplace no)
+			(effects
+				(font
+					(size 1.27 1.27)
+				)
+				(justify left)
+			)
+		)
+		(property "Value" "SW_CAN"
+			(at 361.95 63.4999 90)
+			(show_name no)
+			(do_not_autoplace no)
+			(effects
+				(font
+					(size 1.27 1.27)
+				)
+				(justify left)
+			)
+		)
+		(property "Footprint" "Button_Switch_SMD:SW_SPDT_CK_JS102011SAQN"
+			(at 356.87 62.23 0)
+			(hide yes)
+			(show_name no)
+			(do_not_autoplace no)
+			(effects
+				(font
+					(size 1.27 1.27)
+				)
+			)
+		)
+		(property "Datasheet" ""
+			(at 349.25 62.23 0)
+			(hide yes)
+			(show_name no)
+			(do_not_autoplace no)
+			(effects
+				(font
+					(size 1.27 1.27)
+				)
+			)
+		)
+		(property "Description" "Switch, single pole double throw"
+			(at 356.87 62.23 0)
+			(hide yes)
+			(show_name no)
+			(do_not_autoplace no)
+			(effects
+				(font
+					(size 1.27 1.27)
+				)
+			)
+		)
+		(property "Digi-Key_PN" "401-1999-1-ND"
+			(at 356.87 62.23 90)
+			(hide yes)
+			(show_name no)
+			(do_not_autoplace no)
+			(effects
+				(font
+					(size 1.27 1.27)
+				)
+			)
+		)
+		(pin "1"
+		)
+		(pin "2"
+		)
+		(pin "3"
+		)
+		(instances
+			(project "BIMU_V_1_1"
+				(path "/abeb93ed-b9ef-4503-99a7-3fce380ff294/8f76bfd3-393f-4bde-9261-417b092e4508"
+					(reference "SW203")
+					(unit 1)
+				)

Commit message: Fixer les erreurs commise avec le CAN
Connections:
- net TWAI_CAN_RX: now also U202.1 (TXD); no longer U202.4 (RXD)
- net TWAI_CAN_TX: now also U202.4 (RXD); no longer U202.1 (TXD)
Changed lines of the file:
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@@
 	(global_label "TWAI_CAN_RX"
 		(shape input)
-		(at 308.61 52.07 180)
+		(at 308.61 44.45 180)
 		(fields_autoplaced yes)
 		(effects
@@
 		)
 		(property "Intersheetrefs" "${INTERSHEET_REFS}"
-			(at 293.4086 52.07 0)
+			(at 293.4086 44.45 0)
 			(hide yes)
 			(show_name no)
@@
 	(global_label "TWAI_CAN_TX"
 		(shape input)
-		(at 308.61 44.45 180)
+		(at 308.61 52.07 180)
 		(fields_autoplaced yes)
 		(effects
@@
 		)
 		(property "Intersheetrefs" "${INTERSHEET_REFS}"
-			(at 293.711 44.45 0)
+			(at 293.711 52.07 0)
 			(hide yes)
 			(show_name no)

Commit message: Rajout de Diode pour protégé le USB et la batterie(par short ensemble)
Connections:
- net +5V: no longer J202.A4 (VBUS), J202.A9 (VBUS), J202.B4 (VBUS), J202.B9 (VBUS), J203.7, J204.7
- new net +5V_BAT: J203.7, J204.7
- new net +5V_USB: J202.A4 (VBUS), J202.A9 (VBUS), J202.B4 (VBUS), J202.B9 (VBUS)
Changed lines of the file:
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@@
 	)
 	(junction
+		(at 80.01 38.1)
+		(diameter 0)
+		(color 0 0 0 0)
+	)
+	(junction
 		(at 118.11 88.9)
 		(diameter 0)
@@
 	(wire
 		(pts
+			(xy 80.01 38.1) (xy 92.71 38.1)
+		)
+		(stroke
+			(width 0)
+			(type default)
+		)
+	)
+	(wire
+		(pts
 			(xy 132.08 104.14) (xy 140.97 104.14)
 		)
@@
 	(wire
 		(pts
-			(xy 76.2 38.1) (xy 81.28 38.1)
+			(xy 76.2 38.1) (xy 80.01 38.1)
 		)
 		(stroke
@@
 	(wire
 		(pts
-			(xy 81.28 38.1) (xy 81.28 34.29)
+			(xy 92.71 38.1) (xy 92.71 34.29)
 		)
 		(stroke
@@
 	(symbol
 		(lib_id "power:+5V")
-		(at 81.28 34.29 0)
+		(at 92.71 34.29 0)
 		(unit 1)
 		(body_style 1)
@@
 		(fields_autoplaced yes)
 		(property "Reference" "#PWR0205"
-			(at 81.28 38.1 0)
+			(at 92.71 38.1 0)
 			(hide yes)
 			(show_name no)
@@
 			)
 		)
-		(property "Value" "+5V"
-			(at 81.28 29.21 0)
+		(property "Value" "+5V_USB"
+			(at 95.25 33.0199 0)
 			(show_name no)
 			(do_not_autoplace no)
@@
 					(size 1.27 1.27)
 				)
+				(justify left)
 			)
 		)
 		(property "Footprint" ""
-			(at 81.28 34.29 0)
+			(at 92.71 34.29 0)
 			(hide yes)
 			(show_name no)
@@
 		)
 		(property "Datasheet" ""
-			(at 81.28 34.29 0)
+			(at 92.71 34.29 0)
 			(hide yes)
 			(show_name no)
@@
 		)
 		(property "Description" "Power symbol creates a global label with name \"+5V\""
-			(at 81.28 34.29 0)
+			(at 92.71 34.29 0)
 			(hide yes)
 			(show_name no)
@@
 			)
 		)
-		(property "Value" "+5V"
-			(at 133.35 91.44 90)
+		(property "Value" "+5V_BAT"
+			(at 138.43 94.234 0)
 			(show_name no)
 			(do_not_autoplace no)
@@
 					(unit 1)
 				)
+			)
+		)
+	)
+	(symbol
+		(lib_id "power:PWR_FLAG")
+		(at 80.01 38.1 0)
+		(unit 1)
+		(body_style 1)
+		(exclude_from_sim no)
+		(in_bom yes)
+		(on_board yes)
+		(in_pos_files yes)
+		(dnp no)
+		(fields_autoplaced yes)
+		(property "Reference" "#FLG0203"
+			(at 80.01 36.195 0)
+			(hide yes)
+			(show_name no)
+			(do_not_autoplace no)
+			(effects
+				(font
+					(size 1.27 1.27)
+				)
+			)
+		)
+		(property "Value" "PWR_FLAG"
+			(at 80.01 33.02 0)
+			(show_name no)
+			(do_not_autoplace no)
+			(effects
+				(font
+					(size 1.27 1.27)
+				)
+			)
+		)
+		(property "Footprint" ""
+			(at 80.01 38.1 0)
+			(hide yes)
+			(show_name no)
+			(do_not_autoplace no)
+			(effects
+				(font
+					(size 1.27 1.27)
+				)
+			)
+		)
+		(property "Datasheet" ""
+			(at 80.01 38.1 0)
+			(hide yes)
+			(show_name no)
+			(do_not_autoplace no)
+			(effects
+				(font
+					(size 1.27 1.27)
+				)
+			)
+		)
+		(property "Description" "Special symbol for telling ERC where power comes from"
+			(at 80.01 38.1 0)
+			(hide yes)
+			(show_name no)
+			(do_not_autoplace no)
+			(effects
+				(font
+					(size 1.27 1.27)
+				)
+			)
+		)
+		(pin "1"
+		)
+		(instances
+			(project "BIMU_V_1_1"
+				(path "/abeb93ed-b9ef-4503-99a7-3fce380ff294/8f76bfd3-393f-4bde-9261-417b092e4508"
+					(reference "#FLG0203")
+					(unit 1)
+				)

Commit message: Mise à jour des traces pour TX et RX
Connections:
- net TWAI_CAN_RX: now also U201.5 (GPIO1), U202.4 (RXD); no longer U201.4 (GPIO0), U202.1 (TXD)
- net TWAI_CAN_TX: now also U201.4 (GPIO0), U202.1 (TXD); no longer U201.5 (GPIO1), U202.4 (RXD)
